File: KASM_PCB_REV1.kicad_sch (KiCad schematic)
At the start: 0 parts

Commit message: Add files via upload
Changed lines of the file:
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@@
       (effects (font (size 10 10)) (justify left bottom))
     )
-    (property "Sheetfile" "KASM_PCB_ANALOG.kicad_sch" (at 152.4 186.0046 0)
+    (property "Sheetfile" "KASM_PCB_ANALOG.kicad_sch" (at 152.4 201.93 0)
       (effects (font (size 1.27 1.27)) (justify left top))
     )

Commit message: Add files via upload
Other:
- removed sheet Analog
- removed sheet Connectors
Changed lines of the file:
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@@
-    )
-  )
-  (sheet (at 15.24 114.3) (size 130.81 86.36)
-    (stroke (width 0.1524) (type solid))
-    (fill (color 0 0 0 0.0000))
-    (property "Sheetname" "Connectors" (at 13.97 128.27 0)
-      (effects (font (size 10 10)) (justify left bottom))
-    )
-    (property "Sheetfile" "KASM_PCB_REV1_CONNECTORS.kicad_sch" (at 15.24 201.2446 0)
-      (effects (font (size 1.27 1.27)) (justify left top))
-    )
-    (instances
-      (project "KASM_PCB_REV1"
-        (path "/bcd76057-59fd-41c5-bb52-9bafb2ef74e0" (page "5"))
-      )
-    )
-  )
-  (sheet (at 152.4 114.3) (size 130.81 86.36)
-    (stroke (width 0.1524) (type solid))
-    (fill (color 0 0 0 0.0000))
-    (property "Sheetname" "Analog" (at 152.4 128.27 0)
-      (effects (font (size 10 10)) (justify left bottom))
-    )
-    (property "Sheetfile" "KASM_PCB_ANALOG.kicad_sch" (at 152.4 201.93 0)
-      (effects (font (size 1.27 1.27)) (justify left top))
-    )
-    (instances
-      (project "KASM_PCB_REV1"
-        (path "/bcd76057-59fd-41c5-bb52-9bafb2ef74e0" (page "6"))
-      )
     )
   )
