File: KASM_PCB_REV1.kicad_pcb (KiCad board)
At the start: 2 copper layers, 274 parts, among them J1 Barrel_Jack_Switch, J10 Picoblade, J11 Picoblade, J12 Picoblade, J13 Picoblade, J14 Picoblade, J15 Picoblade, J16 Picoblade, J17 Picoblade, J18 Picoblade, J19 Picoblade, J2 Screw Terminal, J20 Picoblade, J21 Picoblade, J22 Picoblade, J23 Picoblade, J24 Picoblade, J25 Picoblade, J26 Picoblade, J27 Picoblade, J28 Picoblade, J29 Picoblade, J3 Conn_01x02, J30 Picoblade, J31 Picoblade, J32 Picoblade, J33 Picoblade, J34 Picoblade, J4 Conn_01x02, J5 Conn_01x06, J6 Conn_01x05, J7 Conn_01x03, J8 Picoblade, J9 Picoblade, SW1 SW_Push, SW2 SW_Push, U1 TPS5430DDA, U10 STSPIN250, U11 STSPIN250, U12 STSPIN250, U13 STSPIN250, U14 STSPIN250, U15 STSPIN250, U16 STSPIN250, U17 STSPIN250, U18 STSPIN250, U19 STSPIN250, U2 TPS54620, U20 STSPIN250, U21 STSPIN250, U22 STSPIN250, U23 STSPIN250, U24 STSPIN250, U25 STSPIN250, U26 STSPIN250, U27 STSPIN250, U28 STSPIN250, U29 STSPIN250, U3 M24C02-WMN, U30 STSPIN250, U31 STSPIN250, U32 STSPIN250, U33 STSPIN250, U4 TLV9062xD, U6 STM32H750VBTx, U7 STSPIN250, U8 STSPIN250, U9 STSPIN250, Y1 24MHz, 9pF

Commit message: Add files via upload
Parts:
- removed C39, C41, C43, C44, C45, C53, C54, C55, C56, C57, C58, C59, C67, C68, C69, C70, C71, C72, C73, C81, C82, C83, C84, C85, C86: 100nF, Capacitor_SMD:C_0402_1005Metric
- removed C47, C48, C49, C50, C52, C60, C61, C62, C63, C64, C65, C66, C74, C75, C76, C77, C78, C79, C80, C87, C88, C89, C90, C91, C92: 22nF, Capacitor_SMD:C_0402_1005Metric
- removed D3: D_Schottky, Diode_SMD:D_SMA
- removed J10, J11, J12, J14, J15, J16, J17, J18, J19, J20, J21, J22, J23, J24, J25, J26, J27, J28, J29, J30, J31, J32, J33, J34, J9: Picoblade, Connector_Molex:Molex_PicoBlade_53047-0210_1x02_P1.25mm_Vertical
- removed R100, R34, R35, R36, R37, R39, R54, R55, R56, R57, R58, R59, R60, R75, R76, R77, R78, R79, R80, R81, R95, R96, R97, R98, R99: 1k, Resistor_SMD:R_0402_1005Metric
- removed R101, R102, R103, R104, R105, R106, R41, R42, R43, R44, R46, R61, R62, R63, R64, R65, R66, R67, R82, R83, R84, R85, R86, R87, R88: 10k, Resistor_SMD:R_0402_1005Metric
- removed R27, R28, R29, R30, R32, R47, R48, R49, R50, R51, R52, R53, R68, R69, R70, R71, R72, R73, R74, R89, R90, R91, R92, R93, R94: 1.4R, Resistor_SMD:R_1206_3216Metric
- removed U10, U11, U13, U14, U15, U16, U17, U18, U19, U20, U21, U22, U23, U24, U25, U26, U27, U28, U29, U30, U31, U32, U33, U8, U9: STSPIN250, Ultra_librarian:VFQFPN16_STSPIN_STM
- added C100: 100nF, Capacitor_SMD:C_0402_1005Metric, F.Cu at (116.1, 81.5)
- added C101: 22nF, Capacitor_SMD:C_0402_1005Metric, F.Cu at (120.0, 84.7)
- added C102: 100nF, Capacitor_SMD:C_0402_1005Metric, F.Cu at (74.2, 109.6)
- added C103: 22nF, Capacitor_SMD:C_0402_1005Metric, F.Cu at (78.1, 112.7)
- added C104: 100nF, Capacitor_SMD:C_0402_1005Metric, F.Cu at (88.9, 136.8)
- added C105: 22nF, Capacitor_SMD:C_0402_1005Metric, F.Cu at (92.8, 139.9)
- added C106: 100nF, Capacitor_SMD:C_0402_1005Metric, F.Cu at (88.3, 81.5)
- added C107: 22nF, Capacitor_SMD:C_0402_1005Metric, F.Cu at (92.2, 84.7)
- added C108: 100nF, Capacitor_SMD:C_0402_1005Metric, F.Cu at (74.4, 95.8)
- added C109: 22nF, Capacitor_SMD:C_0402_1005Metric, F.Cu at (78.3, 99.0)
- added C110: 100nF, Capacitor_SMD:C_0402_1005Metric, F.Cu at (102.2, 95.8)
- added C111: 22nF, Capacitor_SMD:C_0402_1005Metric, F.Cu at (106.1, 99.0)
- added C112: 100nF, Capacitor_SMD:C_0402_1005Metric, F.Cu at (88.3, 95.8)
- added C113: 22nF, Capacitor_SMD:C_0402_1005Metric, F.Cu at (92.2, 99.0)
- added C114: 100nF, Capacitor_SMD:C_0402_1005Metric, F.Cu at (102.2, 81.5)
- added C115: 22nF, Capacitor_SMD:C_0402_1005Metric, F.Cu at (106.1, 84.7)
- added C116: 100nF, Capacitor_SMD:C_0402_1005Metric, F.Cu at (102.8, 123.1)
- added C117: 22nF, Capacitor_SMD:C_0402_1005Metric, F.Cu at (106.7, 126.2)
- added C118: 100nF, Capacitor_SMD:C_0402_1005Metric, F.Cu at (116.5, 137.1)
- added C119: 22nF, Capacitor_SMD:C_0402_1005Metric, F.Cu at (120.4, 140.2)
- added C120: 100nF, Capacitor_SMD:C_0402_1005Metric, F.Cu at (102.1, 109.6)
- added C121: 22nF, Capacitor_SMD:C_0402_1005Metric, F.Cu at (105.9, 112.7)
- added C122: 100nF, Capacitor_SMD:C_0402_1005Metric, F.Cu at (116.1, 95.8)
- added C123: 22nF, Capacitor_SMD:C_0402_1005Metric, F.Cu at (120.0, 99.0)
- added C124: 100nF, Capacitor_SMD:C_0402_1005Metric, F.Cu at (87.5, 51.2)
- added C125: 22nF, Capacitor_SMD:C_0402_1005Metric, F.Cu at (91.4, 54.4)
- added C126: 100nF, Capacitor_SMD:C_0402_1005Metric, F.Cu at (116.7, 123.1)
- added C127: 22nF, Capacitor_SMD:C_0402_1005Metric, F.Cu at (120.6, 126.2)
- added C128: 100nF, Capacitor_SMD:C_0402_1005Metric, F.Cu at (88.9, 123.1)
- added C129: 22nF, Capacitor_SMD:C_0402_1005Metric, F.Cu at (92.7, 126.2)
- added C130: 100nF, Capacitor_SMD:C_0402_1005Metric, F.Cu at (115.9, 66.3)
- added C131: 22nF, Capacitor_SMD:C_0402_1005Metric, F.Cu at (119.8, 69.4)
- added C132: 100nF, Capacitor_SMD:C_0402_1005Metric, F.Cu at (74.4, 81.5)
- added C133: 22nF, Capacitor_SMD:C_0402_1005Metric, F.Cu at (78.3, 84.7)
- added C134: 100nF, Capacitor_SMD:C_0402_1005Metric, F.Cu at (74.1, 66.3)
- added C135: 22nF, Capacitor_SMD:C_0402_1005Metric, F.Cu at (78.0, 69.4)
- added C136: 100nF, Capacitor_SMD:C_0402_1005Metric, F.Cu at (88.1, 66.3)
- added C137: 22nF, Capacitor_SMD:C_0402_1005Metric, F.Cu at (91.9, 69.4)
- added C138: 100nF, Capacitor_SMD:C_0402_1005Metric, F.Cu at (102.0, 66.3)
- added C139: 22nF, Capacitor_SMD:C_0402_1005Metric, F.Cu at (105.9, 69.4)
- added C140: 100nF, Capacitor_SMD:C_0402_1005Metric, F.Cu at (116.0, 109.6)
- added C141: 22nF, Capacitor_SMD:C_0402_1005Metric, F.Cu at (119.9, 112.7)
- added C142: 100nF, Capacitor_SMD:C_0402_1005Metric, F.Cu at (117.2, 51.2)
- added C143: 22nF, Capacitor_SMD:C_0402_1005Metric, F.Cu at (121.0, 54.3)
- added C93: 100nF, Capacitor_SMD:C_0402_1005Metric, F.Cu at (139.1, 137.9)
- added C94: 100nF, Capacitor_SMD:C_0402_1005Metric, F.Cu at (102.1, 51.2)
- added C95: 22nF, Capacitor_SMD:C_0402_1005Metric, F.Cu at (106.0, 54.3)
- added C96: 100nF, Capacitor_SMD:C_0402_1005Metric, F.Cu at (102.7, 137.0)
- added C97: 22nF, Capacitor_SMD:C_0402_1005Metric, F.Cu at (106.6, 140.2)
- added C98: 100nF, Capacitor_SMD:C_0402_1005Metric, F.Cu at (88.1, 109.6)
- added C99: 22nF, Capacitor_SMD:C_0402_1005Metric, F.Cu at (92.0, 112.7)
- added J35: Picoblade, Connector_Molex:Molex_PicoBlade_53047-0210_1x02_P1.25mm_Vertical, F.Cu at (102.9, 58.1)
- added J36: Picoblade, Connector_Molex:Molex_PicoBlade_53047-0210_1x02_P1.25mm_Vertical, F.Cu at (103.6, 143.9)
- added J37: Picoblade, Connector_Molex:Molex_PicoBlade_53047-0210_1x02_P1.25mm_Vertical, F.Cu at (89.0, 116.5)
- added J38: Picoblade, Connector_Molex:Molex_PicoBlade_53047-0210_1x02_P1.25mm_Vertical, F.Cu at (117.0, 88.4)
- added J39: Picoblade, Connector_Molex:Molex_PicoBlade_53047-0210_1x02_P1.25mm_Vertical, F.Cu at (75.1, 116.5)
- added J40: Picoblade, Connector_Molex:Molex_PicoBlade_53047-0210_1x02_P1.25mm_Vertical, F.Cu at (89.8, 143.7)
- added J41: Picoblade, Connector_Molex:Molex_PicoBlade_53047-0210_1x02_P1.25mm_Vertical, F.Cu at (89.2, 88.4)
- added J42: Picoblade, Connector_Molex:Molex_PicoBlade_53047-0210_1x02_P1.25mm_Vertical, F.Cu at (75.2, 102.7)
- added J43: Picoblade, Connector_Molex:Molex_PicoBlade_53047-0210_1x02_P1.25mm_Vertical, F.Cu at (103.1, 102.7)
- added J44: Picoblade, Connector_Molex:Molex_PicoBlade_53047-0210_1x02_P1.25mm_Vertical, F.Cu at (89.1, 102.7)
- added J45: Picoblade, Connector_Molex:Molex_PicoBlade_53047-0210_1x02_P1.25mm_Vertical, F.Cu at (103.1, 88.4)
- added J46: Picoblade, Connector_Molex:Molex_PicoBlade_53047-0210_1x02_P1.25mm_Vertical, F.Cu at (103.6, 129.9)
- added J47: Picoblade, Connector_Molex:Molex_PicoBlade_53047-0210_1x02_P1.25mm_Vertical, F.Cu at (117.4, 144.0)
- added J48: Picoblade, Connector_Molex:Molex_PicoBlade_53047-0210_1x02_P1.25mm_Vertical, F.Cu at (102.9, 116.5)
- added J49: Picoblade, Connector_Molex:Molex_PicoBlade_53047-0210_1x02_P1.25mm_Vertical, F.Cu at (117.0, 102.7)
- added J50: Picoblade, Connector_Molex:Molex_PicoBlade_53047-0210_1x02_P1.25mm_Vertical, F.Cu at (88.3, 58.1)
- added J51: Picoblade, Connector_Molex:Molex_PicoBlade_53047-0210_1x02_P1.25mm_Vertical, F.Cu at (117.5, 129.9)
- added J52: Picoblade, Connector_Molex:Molex_PicoBlade_53047-0210_1x02_P1.25mm_Vertical, F.Cu at (89.7, 129.9)
- added J53: Picoblade, Connector_Molex:Molex_PicoBlade_53047-0210_1x02_P1.25mm_Vertical, F.Cu at (116.7, 73.1)
- added J54: Picoblade, Connector_Molex:Molex_PicoBlade_53047-0210_1x02_P1.25mm_Vertical, F.Cu at (75.2, 88.4)
- added J55: Picoblade, Connector_Molex:Molex_PicoBlade_53047-0210_1x02_P1.25mm_Vertical, F.Cu at (75.0, 73.1)
- added J56: Picoblade, Connector_Molex:Molex_PicoBlade_53047-0210_1x02_P1.25mm_Vertical, F.Cu at (88.9, 73.1)
- added J57: Picoblade, Connector_Molex:Molex_PicoBlade_53047-0210_1x02_P1.25mm_Vertical, F.Cu at (102.8, 73.1)
- added J58: Picoblade, Connector_Molex:Molex_PicoBlade_53047-0210_1x02_P1.25mm_Vertical, F.Cu at (116.8, 116.5)
- added J59: Picoblade, Connector_Molex:Molex_PicoBlade_53047-0210_1x02_P1.25mm_Vertical, F.Cu at (118.0, 58.1)
- added R108: 1.4R, Resistor_SMD:R_1206_3216Metric, F.Cu at (98.4, 57.0)
- added R109: 1k, Resistor_SMD:R_0402_1005Metric, F.Cu at (106.0, 53.2)
- added R110: 10k, Resistor_SMD:R_0402_1005Metric, F.Cu at (106.0, 52.1)
- added R111: 1.4R, Resistor_SMD:R_1206_3216Metric, F.Cu at (99.0, 142.8)
- added R112: 1k, Resistor_SMD:R_0402_1005Metric, F.Cu at (106.6, 139.0)
- added R113: 10k, Resistor_SMD:R_0402_1005Metric, F.Cu at (106.7, 137.9)
- added R114: 1.4R, Resistor_SMD:R_1206_3216Metric, F.Cu at (84.4, 115.4)
- added R115: 1k, Resistor_SMD:R_0402_1005Metric, F.Cu at (92.0, 111.6)
- added R116: 10k, Resistor_SMD:R_0402_1005Metric, F.Cu at (92.1, 110.5)
- added R117: 1.4R, Resistor_SMD:R_1206_3216Metric, F.Cu at (112.4, 87.3)
- added R118: 1k, Resistor_SMD:R_0402_1005Metric, F.Cu at (120.0, 83.5)
- added R119: 10k, Resistor_SMD:R_0402_1005Metric, F.Cu at (120.0, 82.4)
- added R120: 1.4R, Resistor_SMD:R_1206_3216Metric, F.Cu at (70.5, 115.4)
- added R121: 1k, Resistor_SMD:R_0402_1005Metric, F.Cu at (78.1, 111.6)
- added R122: 10k, Resistor_SMD:R_0402_1005Metric, F.Cu at (78.1, 110.5)
- added R123: 1.4R, Resistor_SMD:R_1206_3216Metric, F.Cu at (85.2, 142.5)
- added R124: 1k, Resistor_SMD:R_0402_1005Metric, F.Cu at (92.8, 138.8)
- added R125: 10k, Resistor_SMD:R_0402_1005Metric, F.Cu at (92.8, 137.7)
- added R126: 1.4R, Resistor_SMD:R_1206_3216Metric, F.Cu at (84.6, 87.3)
- added R127: 1k, Resistor_SMD:R_0402_1005Metric, F.Cu at (92.2, 83.5)
- added R128: 10k, Resistor_SMD:R_0402_1005Metric, F.Cu at (92.2, 82.4)
- added R129: 1.4R, Resistor_SMD:R_1206_3216Metric, F.Cu at (70.7, 101.6)
- added R130: 1k, Resistor_SMD:R_0402_1005Metric, F.Cu at (78.3, 97.8)
- added R131: 10k, Resistor_SMD:R_0402_1005Metric, F.Cu at (78.3, 96.7)
- added R132: 1.4R, Resistor_SMD:R_1206_3216Metric, F.Cu at (98.5, 101.6)
- added R133: 1k, Resistor_SMD:R_0402_1005Metric, F.Cu at (106.1, 97.8)
- added R134: 10k, Resistor_SMD:R_0402_1005Metric, F.Cu at (106.1, 96.7)
- added R135: 1.4R, Resistor_SMD:R_1206_3216Metric, F.Cu at (84.6, 101.6)
- added R136: 1k, Resistor_SMD:R_0402_1005Metric, F.Cu at (92.2, 97.8)
- added R137: 10k, Resistor_SMD:R_0402_1005Metric, F.Cu at (92.2, 96.7)
- added R138: 1.4R, Resistor_SMD:R_1206_3216Metric, F.Cu at (98.5, 87.3)
- added R139: 1k, Resistor_SMD:R_0402_1005Metric, F.Cu at (106.1, 83.5)
- added R140: 10k, Resistor_SMD:R_0402_1005Metric, F.Cu at (106.1, 82.4)
- added R141: 1.4R, Resistor_SMD:R_1206_3216Metric, F.Cu at (99.0, 128.8)
- added R142: 1k, Resistor_SMD:R_0402_1005Metric, F.Cu at (106.7, 125.1)
- added R143: 10k, Resistor_SMD:R_0402_1005Metric, F.Cu at (106.7, 124.0)
- added R144: 1.4R, Resistor_SMD:R_1206_3216Metric, F.Cu at (112.8, 142.9)
- added R145: 1k, Resistor_SMD:R_0402_1005Metric, F.Cu at (120.4, 139.1)
- added R146: 10k, Resistor_SMD:R_0402_1005Metric, F.Cu at (120.4, 138.0)
- added R147: 1.4R, Resistor_SMD:R_1206_3216Metric, F.Cu at (98.3, 115.4)
- added R148: 1k, Resistor_SMD:R_0402_1005Metric, F.Cu at (105.9, 111.6)
- added R149: 10k, Resistor_SMD:R_0402_1005Metric, F.Cu at (106.0, 110.5)
- added R150: 1.4R, Resistor_SMD:R_1206_3216Metric, F.Cu at (112.4, 101.6)
- added R151: 1k, Resistor_SMD:R_0402_1005Metric, F.Cu at (120.0, 97.8)
- added R152: 10k, Resistor_SMD:R_0402_1005Metric, F.Cu at (120.0, 96.7)
- added R153: 1.4R, Resistor_SMD:R_1206_3216Metric, F.Cu at (83.7, 57.0)
- added R154: 1k, Resistor_SMD:R_0402_1005Metric, F.Cu at (91.4, 53.2)
- added R155: 10k, Resistor_SMD:R_0402_1005Metric, F.Cu at (91.4, 52.1)
- added R156: 1.4R, Resistor_SMD:R_1206_3216Metric, F.Cu at (112.9, 128.8)
- added R157: 1k, Resistor_SMD:R_0402_1005Metric, F.Cu at (120.6, 125.1)
- added R158: 10k, Resistor_SMD:R_0402_1005Metric, F.Cu at (120.6, 124.0)
- added R159: 1.4R, Resistor_SMD:R_1206_3216Metric, F.Cu at (85.1, 128.8)
- added R160: 1k, Resistor_SMD:R_0402_1005Metric, F.Cu at (92.7, 125.1)
- added R161: 10k, Resistor_SMD:R_0402_1005Metric, F.Cu at (92.8, 124.0)
- added R162: 1.4R, Resistor_SMD:R_1206_3216Metric, F.Cu at (112.1, 72.0)
- added R163: 1k, Resistor_SMD:R_0402_1005Metric, F.Cu at (119.8, 68.3)
- added R164: 10k, Resistor_SMD:R_0402_1005Metric, F.Cu at (119.8, 67.2)
- added R165: 1.4R, Resistor_SMD:R_1206_3216Metric, F.Cu at (70.7, 87.3)
- added R166: 1k, Resistor_SMD:R_0402_1005Metric, F.Cu at (78.3, 83.5)
- added R167: 10k, Resistor_SMD:R_0402_1005Metric, F.Cu at (78.3, 82.4)
- added R168: 1.4R, Resistor_SMD:R_1206_3216Metric, F.Cu at (70.4, 72.0)
- added R169: 1k, Resistor_SMD:R_0402_1005Metric, F.Cu at (78.0, 68.3)
- added R170: 10k, Resistor_SMD:R_0402_1005Metric, F.Cu at (78.1, 67.2)
- added R171: 1.4R, Resistor_SMD:R_1206_3216Metric, F.Cu at (84.3, 72.0)
- added R172: 1k, Resistor_SMD:R_0402_1005Metric, F.Cu at (91.9, 68.3)
- added R173: 10k, Resistor_SMD:R_0402_1005Metric, F.Cu at (92.0, 67.2)
- added R174: 1.4R, Resistor_SMD:R_1206_3216Metric, F.Cu at (98.2, 72.0)
- added R175: 1k, Resistor_SMD:R_0402_1005Metric, F.Cu at (105.8, 68.3)
- added R176: 10k, Resistor_SMD:R_0402_1005Metric, F.Cu at (105.9, 67.2)
- added R177: 1.4R, Resistor_SMD:R_1206_3216Metric, F.Cu at (112.2, 115.4)
- added R178: 1k, Resistor_SMD:R_0402_1005Metric, F.Cu at (119.8, 111.6)
- added R179: 10k, Resistor_SMD:R_0402_1005Metric, F.Cu at (119.9, 110.5)
- added R180: 1.4R, Resistor_SMD:R_1206_3216Metric, F.Cu at (113.4, 57.0)
- added R181: 1k, Resistor_SMD:R_0402_1005Metric, F.Cu at (121.0, 53.2)
- added R182: 10k, Resistor_SMD:R_0402_1005Metric, F.Cu at (121.1, 52.1)
- added U34: STSPIN250, Ultra_librarian:VFQFPN16_STSPIN_STM, F.Cu at (103.0, 139.8)
- added U35: STSPIN250, Ultra_librarian:VFQFPN16_STSPIN_STM, F.Cu at (88.4, 112.4)
- added U36: STSPIN250, Ultra_librarian:VFQFPN16_STSPIN_STM, F.Cu at (116.4, 84.3)
- added U37: STSPIN250, Ultra_librarian:VFQFPN16_STSPIN_STM, F.Cu at (74.5, 112.4)
- added U38: STSPIN250, Ultra_librarian:VFQFPN16_STSPIN_STM, F.Cu at (89.1, 139.5)
- added U39: STSPIN250, Ultra_librarian:VFQFPN16_STSPIN_STM, F.Cu at (88.5, 84.3)
- added U40: STSPIN250, Ultra_librarian:VFQFPN16_STSPIN_STM, F.Cu at (74.6, 98.6)
- added U41: STSPIN250, Ultra_librarian:VFQFPN16_STSPIN_STM, F.Cu at (102.4, 98.6)
- added U42: STSPIN250, Ultra_librarian:VFQFPN16_STSPIN_STM, F.Cu at (88.5, 98.6)
- added U43: STSPIN250, Ultra_librarian:VFQFPN16_STSPIN_STM, F.Cu at (102.5, 84.3)
- added U44: STSPIN250, Ultra_librarian:VFQFPN16_STSPIN_STM, F.Cu at (103.0, 125.8)
- added U45: STSPIN250, Ultra_librarian:VFQFPN16_STSPIN_STM, F.Cu at (116.8, 139.9)
- added U46: STSPIN250, Ultra_librarian:VFQFPN16_STSPIN_STM, F.Cu at (102.3, 112.4)
- added U47: STSPIN250, Ultra_librarian:VFQFPN16_STSPIN_STM, F.Cu at (116.4, 98.6)
- added U48: STSPIN250, Ultra_librarian:VFQFPN16_STSPIN_STM, F.Cu at (87.7, 54.0)
- added U49: STSPIN250, Ultra_librarian:VFQFPN16_STSPIN_STM, F.Cu at (116.9, 125.8)
- added U5: STSPIN250, Ultra_librarian:VFQFPN16_STSPIN_STM, F.Cu at (74.5, 53.9)
- added U50: STSPIN250, Ultra_librarian:VFQFPN16_STSPIN_STM, F.Cu at (89.1, 125.8)
- added U51: STSPIN250, Ultra_librarian:VFQFPN16_STSPIN_STM, F.Cu at (116.1, 69.0)
- added U52: STSPIN250, Ultra_librarian:VFQFPN16_STSPIN_STM, F.Cu at (74.6, 84.3)
- added U53: STSPIN250, Ultra_librarian:VFQFPN16_STSPIN_STM, F.Cu at (74.4, 69.0)
- added U54: STSPIN250, Ultra_librarian:VFQFPN16_STSPIN_STM, F.Cu at (88.3, 69.0)
- added U55: STSPIN250, Ultra_librarian:VFQFPN16_STSPIN_STM, F.Cu at (102.2, 69.0)
- added U56: STSPIN250, Ultra_librarian:VFQFPN16_STSPIN_STM, F.Cu at (116.2, 112.4)
- added U57: STSPIN250, Ultra_librarian:VFQFPN16_STSPIN_STM, F.Cu at (117.4, 54.0)
- C30: value 10uF -> 4.7uF; footprint Capacitor_SMD:C_1206_3216Metric -> Capacitor_SMD:C_0402_1005Metric
- D1: footprint Diode_SMD:D_SMA -> Diode_SMD:D_SOD-323
- moved C34 132.2 mm to (132.3, 74.1), turned to 90 degrees
- moved C33 129.6 mm to (134.4, 72.2), turned to 180 degrees
- moved C30 125.5 mm to (137.2, 77.6), turned to -90 degrees
- moved C29 123.5 mm to (138.3, 77.6), turned to 90 degrees
- moved C27 122.4 mm to (141.4, 63.8), turned to 180 degrees
- moved U7 115.3 mm to (74.7, 125.9)
- moved L3 114.8 mm to (132.9, 77.9)
- moved Y1 113.5 mm to (134.5, 74.2)
- moved J2 111.8 mm to (174.5, 118.6)
- moved C35 111.4 mm to (152.3, 84.1), turned to -90 degrees
- moved C36 109.2 mm to (157.4, 69.6)
- moved J8 108.6 mm to (75.3, 130.0), turned to 180 degrees
- moved R15 103.1 mm to (137.5, 74.3)
- moved R12 102.2 mm to (135.6, 78.2), turned to 180 degrees
- moved J1 101.2 mm to (166.6, 137.0), turned to 90 degrees
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Connections:
- C30 pad 1: /MCU/VREF+ -> GND
- C30 pad 2: GND -> /MCU/VREF+
- R31 pad 1: Net-(U12-SENSEA) -> Net-(U5-SENSEA)
- R38 pad 1: Net-(U12-TOFF) -> Net-(U5-TOFF)
- R45 pad 1: Net-(U12-TOFF) -> Net-(U5-TOFF)
- U12 pad 1: HRTIM_CHB1_PHASE -> HRTIM_CHC1_PHASE
- U12 pad 10: Net-(J13-Pin_1) -> Net-(J35-Pin_1)
- U12 pad 11: /Drivers/REF -> /Drivers/HRTIM_CHC1/REF
- U12 pad 13: DRIVER_ENABLE -> /Drivers/HRTIM_CHC1/EN
- U12 pad 2: HRTIM_CHB1 -> HRTIM_CHC1
- U12 pad 3: Net-(J13-Pin_1) -> Net-(J35-Pin_1)
- U12 pad 5: Net-(J13-Pin_2) -> Net-(J35-Pin_2)
- U12 pad 8: Net-(J13-Pin_2) -> Net-(J35-Pin_2)
- U7 pad 1: HRTIM_CHC1_PHASE -> HRTIM_CHD1_PHASE
- U7 pad 11: /Drivers/REF -> /Drivers/HRTIM_CHD1/REF
- U7 pad 13: DRIVER_ENABLE -> /Drivers/HRTIM_CHD1/EN
- U7 pad 2: HRTIM_CHC1 -> HRTIM_CHD1
Routing:
- net GND: track 0.00 -> 133.7 mm, vias 0 -> 143
- net +1V8: track 0.00 -> 91.0 mm, vias 0 -> 58
- net Net-(J59-Pin_1): track 0.00 -> 21.8 mm, vias 0 -> 4
- net Net-(J35-Pin_1): track 0.00 -> 21.8 mm, vias 0 -> 4
- net Net-(U57-SENSEA): track 0.00 -> 14.5 mm, vias 0 -> 4
- net Net-(U12-SENSEA): track 0.00 -> 14.5 mm, vias 0 -> 4
- net Net-(J35-Pin_2): track 0.00 -> 13.6 mm
- net Net-(J59-Pin_2): track 0.00 -> 13.6 mm
- net Net-(J57-Pin_1): track 0.00 -> 10.9 mm, vias 0 -> 2
- net Net-(J41-Pin_1): track 0.00 -> 10.9 mm, vias 0 -> 2
- net Net-(J50-Pin_1): track 0.00 -> 10.9 mm, vias 0 -> 2
- net Net-(J45-Pin_1): track 0.00 -> 10.9 mm, vias 0 -> 2
- net Net-(J51-Pin_1): track 0.00 -> 10.9 mm, vias 0 -> 2
- net Net-(J53-Pin_1): track 0.00 -> 10.9 mm, vias 0 -> 2
- net Net-(J36-Pin_1): track 0.00 -> 10.9 mm, vias 0 -> 2
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- added copper zone on F.Cu, net GND
Other:
- board outline added: 115.8 x 104.1 mm
- copper layers 2 -> 4
- board text added: "+ -"
- board text added: "CAP SENSOR 1"
- board text added: "CAP SENSOR 2"

Commit message: Add files via upload
Parts:
- added C39: 100nF, Capacitor_SMD:C_0402_1005Metric, F.Cu at (165.6, 114.3)
- added C41: 4.7uF, Capacitor_SMD:C_0402_1005Metric, F.Cu at (166.9, 114.3)
- added C43: 4.7uF, Capacitor_SMD:C_0402_1005Metric, F.Cu at (165.4, 137.9)
- added C44: 100nF, Capacitor_SMD:C_0402_1005Metric, F.Cu at (166.5, 137.9)
- added FB1: FerriteBead_Small, Inductor_SMD:L_0805_2012Metric, F.Cu at (163.1, 113.3)
- added FB2: FerriteBead_Small, Inductor_SMD:L_0805_2012Metric, F.Cu at (162.8, 136.8)
- added H1: MountingHole_Pad, MountingHole:MountingHole_3.2mm_M3_DIN965_Pad, F.Cu at (68.6, 49.5)
- added H2: MountingHole_Pad, MountingHole:MountingHole_3.2mm_M3_DIN965_Pad, F.Cu at (68.6, 146.1)
- added H3: MountingHole_Pad, MountingHole:MountingHole_3.2mm_M3_DIN965_Pad, F.Cu at (176.5, 49.5)
- added H4: MountingHole_Pad, MountingHole:MountingHole_3.2mm_M3_DIN965_Pad, F.Cu at (176.5, 146.1)
- moved J3 36.2 mm to (175.9, 103.7), turned to 0 degrees
- moved C9 28.6 mm to (158.2, 140.4), turned to -90 degrees
- moved J4 25.2 mm to (175.9, 90.8), turned to 0 degrees
- moved C10 23.5 mm to (155.7, 140.4), turned to -90 degrees
- moved C17 22.9 mm to (133.1, 142.8), turned to 180 degrees
- moved R7 21.9 mm to (137.0, 129.9), turned to 0 degrees
- moved C16 21.9 mm to (133.1, 140.5), turned to 180 degrees
- moved C14 21.8 mm to (133.1, 138.1), turned to 180 degrees
- moved R5 21.8 mm to (154.6, 137.0), turned to 180 degrees
- moved C6 20.9 mm to (156.0, 106.8)
- moved R10 19.5 mm to (139.1, 129.9), turned to 0 degrees
- moved C15 19.3 mm to (136.8, 145.2), turned to 0 degrees
- moved C11 18.5 mm to (153.1, 140.4), turned to -90 degrees
- moved C7 17.8 mm to (139.9, 106.2)
- moved R8 17.8 mm to (152.6, 137.0), turned to 180 degrees
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Connections:
- C10 pad 1: +12V -> Net-(D2-A)
- C11 pad 1: +12V -> Net-(D2-A)
- C2 pad 1: +12V -> Net-(U1-VIN)
- C3 pad 1: +12V -> Net-(U1-VIN)
- C4 pad 1: +12V -> Net-(U1-VIN)
- C5 pad 1: +12V -> Net-(U1-VIN)
- C6 pad 1: +3V3 -> +3.3V
- C7 pad 1: +3V3 -> +3.3V
- C8 pad 1: +12V -> Net-(D2-A)
- C9 pad 1: +12V -> Net-(D2-A)
- C93 pad 1: +12V -> Net-(D2-A)
- D2 pad 2: +12V -> Net-(D2-A)
- L1 pad 2: +3V3 -> +3.3V
- R1 pad 1: +12V -> Net-(U1-VIN)
- R2 pad 1: +3V3 -> +3.3V
- R5 pad 1: +12V -> Net-(D2-A)
- U1 pad 7: +12V -> Net-(U1-VIN)
- U2 pad 4: +12V -> Net-(D2-A)
- U2 pad 5: +12V -> Net-(D2-A)
- U2 pad 6: +12V -> Net-(D2-A)
- U6 pad 71: HRTIM_CHD2 -> unconnected-(U6-PA12-Pad71)
Routing:
- net GND: track 133.7 -> 296.2 mm, vias 143 -> 208
- net HRTIM_CHB1: track 0.00 -> 105.5 mm, vias 0 -> 2
- net HRTIM_CHB1_PHASE: track 0.00 -> 89.3 mm, vias 0 -> 2
- net SPI2_MOSI: track 0.00 -> 50.9 mm, vias 0 -> 2
- net SPI2_MISO: track 0.00 -> 35.9 mm
- net ADC1_INP5: track 0.00 -> 35.0 mm
- net +3.3V: track 0.00 -> 29.5 mm, vias 0 -> 14
- net /MCU/CAP_SENSOR_RET_1: track 0.00 -> 24.2 mm
- net ADC1_INP4: track 0.00 -> 23.8 mm
- net SPI2_NSS: track 0.00 -> 23.6 mm
- net SPI2_SCK: track 0.00 -> 21.4 mm, vias 0 -> 2
- net Net-(D2-A): track 0.00 -> 21.2 mm
- net /MCU/CAP_SENSOR_OUT_1: track 0.00 -> 21.1 mm
- net UART4_RX: track 0.00 -> 20.6 mm, vias 0 -> 1
- net Net-(U1-EN): track 1.04 -> 19.9 mm
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- added copper zone on F.Cu, net +12V
- added copper zone on F.Cu, net +1V8
- added copper zone on In2.Cu, net +1V8
- added copper zone on F.Cu, net +3.3V
- added copper zone on In2.Cu, net +3.3V
- added copper zone on In1.Cu, net GND
- added copper zone on F.Cu, net Net-(C12-Pad2)
- added copper zone on F.Cu, net Net-(D1-K)
- added copper zone on F.Cu, net Net-(D2-A)
- added copper zone on F.Cu, net Net-(U1-VIN)
Other:
- board text added: "+"
- board text added: "-"
- board text removed: "+ -"

Commit message: Add files via upload
Parts:
- moved C37 7.87 mm to (125.5, 97.6)
- moved R23 7.87 mm to (125.5, 95.5)
- moved C2 6.12 mm to (151.5, 121.4)
- moved C3 6.12 mm to (154.1, 121.4)
- moved C4 6.12 mm to (156.7, 121.4)
- moved C41 6.12 mm to (166.8, 120.4)
- moved C5 6.12 mm to (149.6, 121.3)
- moved C6 6.12 mm to (155.9, 112.9)
- moved L1 6.12 mm to (148.0, 113.5)
- moved R4 6.12 mm to (136.0, 121.1)
- moved U1 6.12 mm to (145.1, 121.3)
- moved C1 6.12 mm to (142.4, 117.4)
- moved C39 6.12 mm to (165.6, 120.4)
- moved C7 6.12 mm to (139.9, 112.3)
- moved D1 6.12 mm to (146.8, 117.5)
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Routing:
- net TIM8_CH4: track 0.00 -> 126.5 mm, vias 0 -> 6
- net TIM8_CH4_PHASE: track 0.00 -> 110.7 mm, vias 0 -> 6
- net HRTIM_CHC1_PHASE: track 0.00 -> 99.5 mm, vias 0 -> 4
- net TIM14_CH1: track 0.00 -> 97.5 mm, vias 0 -> 6
- net TIM14_CH1_PHASE: track 0.00 -> 96.8 mm, vias 0 -> 6
- net TIM13_CH1_PHASE: track 0.00 -> 91.1 mm, vias 0 -> 6
- net HRTIM_CHC1: track 0.00 -> 85.9 mm, vias 0 -> 4
- net TIM13_CH1: track 0.00 -> 82.9 mm, vias 0 -> 4
- net TIM15_CH1_PHASE: track 0.00 -> 78.4 mm, vias 0 -> 6
- net TIM4_CH3: track 0.00 -> 64.4 mm, vias 0 -> 4
- net HRTIM_CHA1: track 0.00 -> 56.8 mm, vias 0 -> 4
- net TIM15_CH1: track 0.00 -> 54.7 mm, vias 0 -> 4
- net TIM4_CH3_PHASE: track 0.00 -> 51.5 mm, vias 0 -> 4
- net SPI2_MOSI: track 50.9 -> 0.00 mm, vias 2 -> 0
- net HRTIM_CHA1_PHASE: track 0.00 -> 45.5 mm, vias 0 -> 4
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
Commit message: Add files via upload
Routing:
- net HRTIM_CHC2: track 0.00 -> 126.9 mm, vias 0 -> 6
- net HRTIM_CHC2_PHASE: track 0.00 -> 95.7 mm, vias 0 -> 6
- net TIM5_CH2_PHASE: track 0.00 -> 86.3 mm, vias 0 -> 4
- net TIM4_CH1: track 0.00 -> 86.1 mm, vias 0 -> 6
- net TIM4_CH1_PHASE: track 0.00 -> 78.9 mm, vias 0 -> 6
- net TIM5_CH2: track 0.00 -> 76.6 mm, vias 0 -> 2
- net TIM2_CH1: track 0.00 -> 33.9 mm, vias 0 -> 2
