File: KASM_PCB_REV1.kicad_pcb (KiCad board)
At the start: 4 copper layers, 115.8 x 104.1 mm, 284 parts, among them J1 Barrel_Jack_Switch, J13 Picoblade, J2 Screw Terminal, J3 Conn_01x02, J35 Picoblade, J36 Picoblade, J37 Picoblade, J38 Picoblade, J39 Picoblade, J4 Conn_01x02, J40 Picoblade, J41 Picoblade, J42 Picoblade, J43 Picoblade, J44 Picoblade, J45 Picoblade, J46 Picoblade, J47 Picoblade, J48 Picoblade, J49 Picoblade, J5 Conn_01x06, J50 Picoblade, J51 Picoblade, J52 Picoblade, J53 Picoblade, J54 Picoblade, J55 Picoblade, J56 Picoblade, J57 Picoblade, J58 Picoblade, J59 Picoblade, J6 Conn_01x05, J7 Conn_01x03, J8 Picoblade, SW1 SW_Push, SW2 SW_Push, U1 TPS5430DDA, U12 STSPIN250, U2 TPS54620, U3 M24C02-WMN, U34 STSPIN250, U35 STSPIN250, U36 STSPIN250, U37 STSPIN250, U38 STSPIN250, U39 STSPIN250, U4 TLV9062xD, U40 STSPIN250, U41 STSPIN250, U42 STSPIN250, U43 STSPIN250, U44 STSPIN250, U45 STSPIN250, U46 STSPIN250, U47 STSPIN250, U48 STSPIN250, U49 STSPIN250, U5 STSPIN250, U50 STSPIN250, U51 STSPIN250, U52 STSPIN250, U53 STSPIN250, U54 STSPIN250, U55 STSPIN250, U56 STSPIN250, U57 STSPIN250, U6 STM32H750VBTx, U7 STSPIN250, Y1 24MHz, 9pF

Commit message: Add files via upload
Parts:
- moved C38 7.61 mm to (134.4, 99.8)
- moved R25 7.61 mm to (133.3, 99.8)
- moved R24 7.61 mm to (134.4, 97.7)
- moved C37 2.02 mm to (125.2, 99.6)
- moved R23 2.02 mm to (125.2, 97.5)
Connections:
- net /Drivers/REF renamed REF
- U6 pad 71: unconnected-(U6-PA12-Pad71) -> HRTIM_CHD2
Routing:
- net HRTIM_CHA2_PHASE: track 0.00 -> 168.0 mm, vias 0 -> 4
- net HRTIM_CHA2: track 0.00 -> 149.7 mm, vias 0 -> 4
- net HRTIM_CHD2: track 0.00 -> 136.6 mm, vias 0 -> 4
- net LPTIM1_OUT: track 0.00 -> 131.4 mm, vias 0 -> 6
- net LPTIM1_OUT_PHASE: track 0.00 -> 127.1 mm, vias 0 -> 6
- net HRTIM_CHD2_PHASE: track 0.00 -> 117.0 mm, vias 0 -> 4
- net TIM4_CH2: track 0.00 -> 113.4 mm, vias 0 -> 6
- net TIM15_CH2_PHASE: track 0.00 -> 108.3 mm, vias 0 -> 6
- net TIM4_CH2_PHASE: track 0.00 -> 105.7 mm, vias 0 -> 6
- net TIM1_CH3: track 0.00 -> 105.1 mm, vias 0 -> 4
- net TIM1_CH3_PHASE: track 0.00 -> 102.4 mm, vias 0 -> 4
- net TIM1_CH4: track 0.00 -> 90.6 mm, vias 0 -> 4
- net TIM1_CH4_PHASE: track 0.00 -> 90.0 mm, vias 0 -> 4
- net TIM15_CH2: track 0.00 -> 89.6 mm, vias 0 -> 4
- net TIM16_CH1_PHASE: track 0.00 -> 89.0 mm, vias 0 -> 6
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
Commit message: Add files via upload
Parts:
- moved C36 1.02 mm to (158.4, 69.6)
Routing:
- net HRTIM_CHB2: track 0.00 -> 166.9 mm, vias 0 -> 6
- net HRTIM_CHD1: track 0.00 -> 160.8 mm, vias 0 -> 6
- net HRTIM_CHD1_PHASE: track 0.00 -> 151.3 mm, vias 0 -> 6
- net HRTIM_CHB2_PHASE: track 0.00 -> 147.0 mm, vias 0 -> 8
- net TIM1_CH1_PHASE: track 0.00 -> 121.4 mm, vias 0 -> 8
- net TIM1_CH1: track 0.00 -> 116.2 mm, vias 0 -> 6
- net TIM4_CH4: track 0.00 -> 111.4 mm, vias 0 -> 6
- net TIM4_CH4_PHASE: track 0.00 -> 97.2 mm, vias 0 -> 6
- net DEBUG_JTDO-SWO: track 0.00 -> 93.4 mm, vias 0 -> 4
- net /MCU/NRST: track 0.00 -> 65.3 mm, vias 0 -> 5
- net SPI2_MOSI: track 0.00 -> 53.7 mm, vias 0 -> 3
- net /MCU/BOOT0: track 0.00 -> 51.4 mm, vias 0 -> 2
- net SPI2_MISO: track 0.00 -> 41.0 mm, vias 0 -> 1
- net DEBUG_JTMS-SWDIO: track 0.00 -> 32.4 mm, vias 0 -> 4
- net SPI2_SCK: track 0.00 -> 32.1 mm, vias 0 -> 3
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
Commit message: Add files via upload
Parts:
- moved R124 0.65 mm to (93.4, 138.8)
- moved C105 0.65 mm to (93.5, 139.9)
- moved R125 0.65 mm to (93.5, 137.7)
- moved R163 0.61 mm to (120.4, 68.3)
- moved C131 0.61 mm to (120.4, 69.4)
- moved R164 0.61 mm to (120.4, 67.2)
- moved C123 0.61 mm to (120.6, 99.0)
- moved R151 0.61 mm to (120.6, 97.8)
- moved R152 0.61 mm to (120.7, 96.7)
- moved C101 0.60 mm to (120.6, 84.7)
- moved R118 0.60 mm to (120.6, 83.5)
- moved R119 0.60 mm to (120.7, 82.4)
- moved C143 0.60 mm to (128.8, 54.5)
- moved R182 0.60 mm to (128.8, 52.3)
- moved R181 0.60 mm to (128.7, 53.4)
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Connections:
- U12 pad 11: /Drivers/HRTIM_CHC1/REF -> REF
- U34 pad 11: /Drivers/TIM1_CH1/REF -> REF
- U35 pad 11: /Drivers/TIM1_CH3/REF -> REF
- U36 pad 11: /Drivers/TIM2_CH1/REF -> REF
- U37 pad 11: /Drivers/HRTIM_CHA2/REF -> REF
- U38 pad 11: /Drivers/HRTIM_CHB2/REF -> REF
- U39 pad 11: /Drivers/HRTIM_CHC2/REF -> REF
- U40 pad 11: /Drivers/HRTIM_CHD2/REF -> REF
- U41 pad 11: /Drivers/TIM1_CH2/REF -> REF
- U42 pad 11: /Drivers/TIM1_CH4/REF -> REF
- U43 pad 11: /Drivers/TIM4_CH1/REF -> REF
- U44 pad 11: /Drivers/TIM4_CH2/REF -> REF
- U45 pad 11: /Drivers/TIM4_CH4/REF -> REF
- U46 pad 11: /Drivers/TIM5_CH3/REF -> REF
- U47 pad 11: /Drivers/TIM12_CH2/REF -> REF
- U48 pad 11: /Drivers/TIM14_CH1/REF -> REF
- U49 pad 11: /Drivers/TIM15_CH2/REF -> REF
- U5 pad 11: /Drivers/HRTIM_CHB1/REF -> REF
- U50 pad 11: /Drivers/LPTIM1_OUT/REF -> REF
- U51 pad 11: /Drivers/TIM4_CH3/REF -> REF
- U52 pad 11: /Drivers/TIM5_CH2/REF -> REF
- U53 pad 11: /Drivers/TIM8_CH4/REF -> REF
- U54 pad 11: /Drivers/TIM13_CH1/REF -> REF
- U55 pad 11: /Drivers/TIM15_CH1/REF -> REF
- U56 pad 11: /Drivers/TIM16_CH1/REF -> REF
- U57 pad 11: /Drivers/HRTIM_CHA1/REF -> REF
- U7 pad 11: /Drivers/HRTIM_CHD1/REF -> REF
Routing:
- net REF: track 2.15 -> 424.0 mm, vias 0 -> 35
- net Net-(J59-Pin_1): track 21.8 -> 12.5 mm, vias 4 -> 2
- net SPI2_SCK: track 32.1 -> 34.6 mm, vias 3 -> 5
- net Net-(J35-Pin_1): track 21.8 -> 19.6 mm, vias 4 -> 2
- net Net-(U12-TOFF): track 5.61 -> 3.44 mm
- net Net-(C143-Pad1): track 2.26 -> 1.09 mm
- net Net-(C95-Pad1): track 2.26 -> 1.17 mm
- net Net-(U57-TOFF): track 5.61 -> 4.70 mm
- net Net-(U51-TOFF): track 2.81 -> 3.49 mm
- net Net-(U38-TOFF): track 2.81 -> 3.48 mm
- net Net-(U36-TOFF): track 2.81 -> 3.48 mm
- net Net-(U55-TOFF): track 2.81 -> 3.45 mm
- net Net-(U47-TOFF): track 2.81 -> 3.44 mm
- net Net-(U37-TOFF): track 2.81 -> 3.42 mm
- net Net-(U49-TOFF): track 2.81 -> 3.40 mm
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