File: KASM_PCB_REV1.kicad_pcb (KiCad board)
At the start: 4 copper layers, 115.8 x 104.1 mm, 284 parts, among them J1 Barrel_Jack_Switch, J13 Picoblade, J2 Screw Terminal, J3 Conn_01x02, J35 Picoblade, J36 Picoblade, J37 Picoblade, J38 Picoblade, J39 Picoblade, J4 Conn_01x02, J40 Picoblade, J41 Picoblade, J42 Picoblade, J43 Picoblade, J44 Picoblade, J45 Picoblade, J46 Picoblade, J47 Picoblade, J48 Picoblade, J49 Picoblade, J5 Conn_01x06, J50 Picoblade, J51 Picoblade, J52 Picoblade, J53 Picoblade, J54 Picoblade, J55 Picoblade, J56 Picoblade, J57 Picoblade, J58 Picoblade, J59 Picoblade, J6 Conn_01x05, J7 Conn_01x03, J8 Picoblade, SW1 SW_Push, SW2 SW_Push, U1 TPS5430DDA, U12 STSPIN250, U2 TPS54620, U3 M24C02-WMN, U34 STSPIN250, U35 STSPIN250, U36 STSPIN250, U37 STSPIN250, U38 STSPIN250, U39 STSPIN250, U4 TLV9062xD, U40 STSPIN250, U41 STSPIN250, U42 STSPIN250, U43 STSPIN250, U44 STSPIN250, U45 STSPIN250, U46 STSPIN250, U47 STSPIN250, U48 STSPIN250, U49 STSPIN250, U5 STSPIN250, U50 STSPIN250, U51 STSPIN250, U52 STSPIN250, U53 STSPIN250, U54 STSPIN250, U55 STSPIN250, U56 STSPIN250, U57 STSPIN250, U6 STM32H750VBTx, U7 STSPIN250, Y1 24MHz, 9pF

Commit message: Add files via upload
Parts:
- added C45: 100nF, Capacitor_SMD:C_0402_1005Metric, F.Cu at (208.2, 92.6)
- added C47: 100nF, Capacitor_SMD:C_0402_1005Metric, F.Cu at (222.9, 74.7)
- added C48: 100nF, Capacitor_SMD:C_0402_1005Metric, F.Cu at (227.8, 74.7)
- added C49: 100nF, Capacitor_SMD:C_0402_1005Metric, F.Cu at (213.1, 80.7)
- added C50: 100nF, Capacitor_SMD:C_0402_1005Metric, F.Cu at (208.2, 68.8)
- added C52: 100nF, Capacitor_SMD:C_0402_1005Metric, F.Cu at (208.2, 86.6)
- added C53: 100nF, Capacitor_SMD:C_0402_1005Metric, F.Cu at (222.9, 86.6)
- added C54: 100nF, Capacitor_SMD:C_0402_1005Metric, F.Cu at (218.0, 74.7)
- added C55: 100nF, Capacitor_SMD:C_0402_1005Metric, F.Cu at (213.1, 74.7)
- added C56: 100nF, Capacitor_SMD:C_0402_1005Metric, F.Cu at (213.1, 68.8)
- added C57: 100nF, Capacitor_SMD:C_0402_1005Metric, F.Cu at (213.1, 86.6)
- added C58: 100nF, Capacitor_SMD:C_0402_1005Metric, F.Cu at (218.0, 86.6)
- added C59: 100nF, Capacitor_SMD:C_0402_1005Metric, F.Cu at (218.0, 80.7)
- added C60: 100nF, Capacitor_SMD:C_0402_1005Metric, F.Cu at (203.2, 74.7)
- added C61: 100nF, Capacitor_SMD:C_0402_1005Metric, F.Cu at (227.8, 68.8)
- added C62: 100nF, Capacitor_SMD:C_0402_1005Metric, F.Cu at (222.9, 68.8)
- added C63: 100nF, Capacitor_SMD:C_0402_1005Metric, F.Cu at (208.2, 74.7)
- added C64: 100nF, Capacitor_SMD:C_0402_1005Metric, F.Cu at (203.2, 86.6)
- added C65: 100nF, Capacitor_SMD:C_0402_1005Metric, F.Cu at (213.1, 92.6)
- added C66: 100nF, Capacitor_SMD:C_0402_1005Metric, F.Cu at (227.8, 80.7)
- added C67: 100nF, Capacitor_SMD:C_0402_1005Metric, F.Cu at (203.2, 68.8)
- added C68: 100nF, Capacitor_SMD:C_0402_1005Metric, F.Cu at (222.9, 80.7)
- added C69: 100nF, Capacitor_SMD:C_0402_1005Metric, F.Cu at (208.2, 80.7)
- added C70: 100nF, Capacitor_SMD:C_0402_1005Metric, F.Cu at (218.0, 92.6)
- added C71: 100nF, Capacitor_SMD:C_0402_1005Metric, F.Cu at (203.2, 80.7)
- added C72: 100nF, Capacitor_SMD:C_0402_1005Metric, F.Cu at (203.2, 92.6)
- added R27: 10k, Resistor_SMD:R_0402_1005Metric, F.Cu at (208.2, 90.6)
- added R28: 10k, Resistor_SMD:R_0402_1005Metric, F.Cu at (222.9, 72.7)
- added R29: 10k, Resistor_SMD:R_0402_1005Metric, F.Cu at (227.8, 72.7)
- added R30: 10k, Resistor_SMD:R_0402_1005Metric, F.Cu at (213.1, 78.7)
- added R32: 10k, Resistor_SMD:R_0402_1005Metric, F.Cu at (208.2, 66.8)
- added R34: 10k, Resistor_SMD:R_0402_1005Metric, F.Cu at (208.2, 84.7)
- added R35: 10k, Resistor_SMD:R_0402_1005Metric, F.Cu at (222.9, 84.7)
- added R36: 10k, Resistor_SMD:R_0402_1005Metric, F.Cu at (218.0, 72.7)
- added R37: 10k, Resistor_SMD:R_0402_1005Metric, F.Cu at (213.1, 72.7)
- added R39: 10k, Resistor_SMD:R_0402_1005Metric, F.Cu at (213.1, 66.8)
- added R41: 10k, Resistor_SMD:R_0402_1005Metric, F.Cu at (213.1, 84.7)
- added R42: 10k, Resistor_SMD:R_0402_1005Metric, F.Cu at (218.0, 84.7)
- added R43: 10k, Resistor_SMD:R_0402_1005Metric, F.Cu at (218.0, 78.7)
- added R44: 10k, Resistor_SMD:R_0402_1005Metric, F.Cu at (203.3, 72.7)
- added R46: 10k, Resistor_SMD:R_0402_1005Metric, F.Cu at (227.8, 66.8)
- added R47: 10k, Resistor_SMD:R_0402_1005Metric, F.Cu at (222.9, 66.8)
- added R48: 10k, Resistor_SMD:R_0402_1005Metric, F.Cu at (208.2, 72.7)
- added R49: 10k, Resistor_SMD:R_0402_1005Metric, F.Cu at (203.3, 84.7)
- added R50: 10k, Resistor_SMD:R_0402_1005Metric, F.Cu at (213.1, 90.6)
- added R51: 10k, Resistor_SMD:R_0402_1005Metric, F.Cu at (227.8, 78.7)
- added R52: 10k, Resistor_SMD:R_0402_1005Metric, F.Cu at (203.3, 66.8)
- added R53: 10k, Resistor_SMD:R_0402_1005Metric, F.Cu at (222.9, 78.7)
- added R54: 10k, Resistor_SMD:R_0402_1005Metric, F.Cu at (208.2, 78.7)
- added R55: 10k, Resistor_SMD:R_0402_1005Metric, F.Cu at (218.0, 90.6)
- added R56: 10k, Resistor_SMD:R_0402_1005Metric, F.Cu at (203.3, 78.7)
- added R57: 10k, Resistor_SMD:R_0402_1005Metric, F.Cu at (203.3, 90.6)
- moved R23 97.7 mm to (218.0, 66.8), turned to 0 degrees
- moved C37 97.7 mm to (218.0, 68.8), turned to 0 degrees
Connections:
- C37 pad 1: DRIVER_ENABLE -> /Drivers/HRTIM_CHA1/EN
- R23 pad 2: DRIVER_ENABLE -> /Drivers/HRTIM_CHA1/EN
Routing:
- net REF: track 424.0 -> 441.9 mm, vias 35 -> 38
- net Net-(J59-Pin_1): track 12.5 -> 14.8 mm
- net DRIVER_ENABLE: track 1.04 -> 0.00 mm
- net +1V8: track 97.9 -> 97.0 mm, vias 67 -> 66
- net GND: track 315.6 -> 314.8 mm, vias 216 -> 215
- net +3.3V: vias 20 -> 35
