File: KASM_PCB_REV1_DRIVERS.kicad_sch (KiCad schematic)
At the start: 167 parts, among them J10 Picoblade, J11 Picoblade, J12 Picoblade, J13 Picoblade, J14 Picoblade, J15 Picoblade, J16 Picoblade, J17 Picoblade, J18 Picoblade, J19 Picoblade, J2 Picoblade, J20 Picoblade, J21 Picoblade, J22 Picoblade, J23 Picoblade, J24 Picoblade, J25 Picoblade, J26 Picoblade, J27 Picoblade, J28 Picoblade, J29 Picoblade, J30 Picoblade, J5 Picoblade, J6 Picoblade, J7 Picoblade, J8 Picoblade, J9 Picoblade, U10 STSPIN250, U11 STSPIN250, U12 STSPIN250, U13 STSPIN250, U14 STSPIN250, U15 STSPIN250, U16 STSPIN250, U17 STSPIN250, U18 STSPIN250, U19 STSPIN250, U2 STSPIN250, U20 STSPIN250, U21 STSPIN250, U22 STSPIN250, U23 STSPIN250, U24 STSPIN250, U25 STSPIN250, U26 STSPIN250, U27 STSPIN250, U28 STSPIN250, U30 STSPIN250, U31 STSPIN250, U32 STSPIN250, U33 STSPIN250, U7 STSPIN250, U8 STSPIN250, U9 STSPIN250

Commit message: Add files via upload
Parts:
- removed C41: 100n, symbol Device:C_Small
- added C19 (x28): 100nF, Capacitor_SMD:C_0402_1005Metric, symbol Device:C_Small
- C38: renamed from C42; value 1u -> 1uF; footprint (none) -> Capacitor_SMD:C_0402_1005Metric; LCSC (none) -> C52923
- C46: renamed from C45; value 22n -> 22nF; footprint (none) -> Capacitor_SMD:C_0402_1005Metric; LCSC (none) -> C1532
- C47: renamed from C46; value 22n -> 22nF; footprint (none) -> Capacitor_SMD:C_0402_1005Metric; LCSC (none) -> C1532
- C48: renamed from C47; value 22n -> 22nF; footprint (none) -> Capacitor_SMD:C_0402_1005Metric; LCSC (none) -> C1532
- C49: renamed from C48; value 22n -> 22nF; footprint (none) -> Capacitor_SMD:C_0402_1005Metric; LCSC (none) -> C1532
- C50: renamed from C49; value 22n -> 22nF; footprint (none) -> Capacitor_SMD:C_0402_1005Metric; LCSC (none) -> C1532
- C51: renamed from C44; value 22n -> 22nF; footprint (none) -> Capacitor_SMD:C_0402_1005Metric; LCSC (none) -> C1532
- C52: renamed from C43; value 22n -> 22nF; footprint (none) -> Capacitor_SMD:C_0402_1005Metric; LCSC (none) -> C1532
- C60: renamed from C55; value 22n -> 22nF; footprint (none) -> Capacitor_SMD:C_0402_1005Metric; LCSC (none) -> C1532
- C61: renamed from C54; value 22n -> 22nF; footprint (none) -> Capacitor_SMD:C_0402_1005Metric; LCSC (none) -> C1532
- C62: renamed from C53; value 22n -> 22nF; footprint (none) -> Capacitor_SMD:C_0402_1005Metric; LCSC (none) -> C1532
- C63: renamed from C52; value 22n -> 22nF; footprint (none) -> Capacitor_SMD:C_0402_1005Metric; LCSC (none) -> C1532
- C64: renamed from C51; value 22n -> 22nF; footprint (none) -> Capacitor_SMD:C_0402_1005Metric; LCSC (none) -> C1532
- C65: renamed from C50; value 22n -> 22nF; footprint (none) -> Capacitor_SMD:C_0402_1005Metric; LCSC (none) -> C1532
- C66: renamed from C56; value 22n -> 22nF; footprint (none) -> Capacitor_SMD:C_0402_1005Metric; LCSC (none) -> C1532
- C74: renamed from C57; value 22n -> 22nF; footprint (none) -> Capacitor_SMD:C_0402_1005Metric; LCSC (none) -> C1532
- C75: renamed from C58; value 22n -> 22nF; footprint (none) -> Capacitor_SMD:C_0402_1005Metric; LCSC (none) -> C1532
- C76: renamed from C59; value 22n -> 22nF; footprint (none) -> Capacitor_SMD:C_0402_1005Metric; LCSC (none) -> C1532
- C77: renamed from C60; value 22n -> 22nF; footprint (none) -> Capacitor_SMD:C_0402_1005Metric; LCSC (none) -> C1532
- C78: renamed from C61; value 22n -> 22nF; footprint (none) -> Capacitor_SMD:C_0402_1005Metric; LCSC (none) -> C1532
- C79: renamed from C62; value 22n -> 22nF; footprint (none) -> Capacitor_SMD:C_0402_1005Metric; LCSC (none) -> C1532
- C80: renamed from C63; value 22n -> 22nF; footprint (none) -> Capacitor_SMD:C_0402_1005Metric; LCSC (none) -> C1532
- C87: renamed from C69; value 22n -> 22nF; footprint (none) -> Capacitor_SMD:C_0402_1005Metric; LCSC (none) -> C1532
- C88: renamed from C68; value 22n -> 22nF; footprint (none) -> Capacitor_SMD:C_0402_1005Metric; LCSC (none) -> C1532
- C89: renamed from C67; value 22n -> 22nF; footprint (none) -> Capacitor_SMD:C_0402_1005Metric; LCSC (none) -> C1532
- C90: renamed from C66; value 22n -> 22nF; footprint (none) -> Capacitor_SMD:C_0402_1005Metric; LCSC (none) -> C1532
- C91: renamed from C65; value 22n -> 22nF; footprint (none) -> Capacitor_SMD:C_0402_1005Metric; LCSC (none) -> C1532
- C92: renamed from C64; value 22n -> 22nF; footprint (none) -> Capacitor_SMD:C_0402_1005Metric; LCSC (none) -> C1532
- R100: renamed from R85; footprint (none) -> Resistor_SMD:R_0402_1005Metric; LCSC (none) -> C11702
- R101: footprint (none) -> Resistor_SMD:R_0402_1005Metric; LCSC (none) -> C25744
- R102: renamed from R98; footprint (none) -> Resistor_SMD:R_0402_1005Metric; LCSC (none) -> C25744
- R103: renamed from R95; footprint (none) -> Resistor_SMD:R_0402_1005Metric; LCSC (none) -> C25744
- R104: renamed from R92; footprint (none) -> Resistor_SMD:R_0402_1005Metric; LCSC (none) -> C25744
- R105: renamed from R89; footprint (none) -> Resistor_SMD:R_0402_1005Metric; LCSC (none) -> C25744
- R106: renamed from R86; footprint (none) -> Resistor_SMD:R_0402_1005Metric; LCSC (none) -> C25744
- R23: renamed from R18; footprint (none) -> Resistor_SMD:R_0402_1005Metric; LCSC (none) -> C25744
- R24: renamed from R21; footprint (none) -> Resistor_SMD:R_0402_1005Metric; LCSC (none) -> C25908
- R25: renamed from R22; footprint (none) -> Resistor_SMD:R_0402_1005Metric; LCSC (none) -> C11702
- R26: renamed from R27; footprint (none) -> Resistor_SMD:R_1206_3216Metric; LCSC C5126235 -> C305315
- R27: renamed from R30; footprint (none) -> Resistor_SMD:R_1206_3216Metric; LCSC C5126235 -> C305315
- R28: renamed from R33; footprint (none) -> Resistor_SMD:R_1206_3216Metric; LCSC C5126235 -> C305315
- R29: renamed from R36; footprint (none) -> Resistor_SMD:R_1206_3216Metric; LCSC C5126235 -> C305315
- R30: renamed from R39; footprint (none) -> Resistor_SMD:R_1206_3216Metric; LCSC C5126235 -> C305315
- R31: renamed from R24; footprint (none) -> Resistor_SMD:R_1206_3216Metric; LCSC C5126235 -> C305315
- R32: renamed from R23; footprint (none) -> Resistor_SMD:R_1206_3216Metric; LCSC C5126235 -> C305315
- R33: renamed from R28; footprint (none) -> Resistor_SMD:R_0402_1005Metric; LCSC (none) -> C11702
- R34: renamed from R31; footprint (none) -> Resistor_SMD:R_0402_1005Metric; LCSC (none) -> C11702
- R35: renamed from R34; footprint (none) -> Resistor_SMD:R_0402_1005Metric; LCSC (none) -> C11702
- R36: renamed from R37; footprint (none) -> Resistor_SMD:R_0402_1005Metric; LCSC (none) -> C11702
- R37: renamed from R40; footprint (none) -> Resistor_SMD:R_0402_1005Metric; LCSC (none) -> C11702
- R38: renamed from R25; footprint (none) -> Resistor_SMD:R_0402_1005Metric; LCSC (none) -> C11702
- R39: renamed from R20; footprint (none) -> Resistor_SMD:R_0402_1005Metric; LCSC (none) -> C11702
- R40: renamed from R29; footprint (none) -> Resistor_SMD:R_0402_1005Metric; LCSC (none) -> C25744
- R41: renamed from R32; footprint (none) -> Resistor_SMD:R_0402_1005Metric; LCSC (none) -> C25744
- R42: renamed from R35; footprint (none) -> Resistor_SMD:R_0402_1005Metric; LCSC (none) -> C25744
- R43: renamed from R38; footprint (none) -> Resistor_SMD:R_0402_1005Metric; LCSC (none) -> C25744
- R44: renamed from R41; footprint (none) -> Resistor_SMD:R_0402_1005Metric; LCSC (none) -> C25744
- R45: renamed from R26; footprint (none) -> Resistor_SMD:R_0402_1005Metric; LCSC (none) -> C25744
- R46: renamed from R19; footprint (none) -> Resistor_SMD:R_0402_1005Metric; LCSC (none) -> C25744
- R47: renamed from R57; footprint (none) -> Resistor_SMD:R_1206_3216Metric; LCSC C5126235 -> C305315
- R48: renamed from R54; footprint (none) -> Resistor_SMD:R_1206_3216Metric; LCSC C5126235 -> C305315
- R49: renamed from R51; footprint (none) -> Resistor_SMD:R_1206_3216Metric; LCSC C5126235 -> C305315
- R50: renamed from R48; footprint (none) -> Resistor_SMD:R_1206_3216Metric; LCSC C5126235 -> C305315
- R51: renamed from R45; footprint (none) -> Resistor_SMD:R_1206_3216Metric; LCSC C5126235 -> C305315
- R52: renamed from R42; footprint (none) -> Resistor_SMD:R_1206_3216Metric; LCSC C5126235 -> C305315
- R53: renamed from R60; footprint (none) -> Resistor_SMD:R_1206_3216Metric; LCSC C5126235 -> C305315
- R54: renamed from R58; footprint (none) -> Resistor_SMD:R_0402_1005Metric; LCSC (none) -> C11702
- R55: footprint (none) -> Resistor_SMD:R_0402_1005Metric; LCSC (none) -> C11702
- R56: renamed from R52; footprint (none) -> Resistor_SMD:R_0402_1005Metric; LCSC (none) -> C11702
- R57: renamed from R49; footprint (none) -> Resistor_SMD:R_0402_1005Metric; LCSC (none) -> C11702
- R58: renamed from R46; footprint (none) -> Resistor_SMD:R_0402_1005Metric; LCSC (none) -> C11702
- R59: renamed from R43; footprint (none) -> Resistor_SMD:R_0402_1005Metric; LCSC (none) -> C11702
- R60: renamed from R61; footprint (none) -> Resistor_SMD:R_0402_1005Metric; LCSC (none) -> C11702
- R61: renamed from R59; footprint (none) -> Resistor_SMD:R_0402_1005Metric; LCSC (none) -> C25744
- R62: renamed from R56; footprint (none) -> Resistor_SMD:R_0402_1005Metric; LCSC (none) -> C25744
- R63: renamed from R53; footprint (none) -> Resistor_SMD:R_0402_1005Metric; LCSC (none) -> C25744
- R64: renamed from R50; footprint (none) -> Resistor_SMD:R_0402_1005Metric; LCSC (none) -> C25744
- R65: renamed from R47; footprint (none) -> Resistor_SMD:R_0402_1005Metric; LCSC (none) -> C25744
- R66: renamed from R44; footprint (none) -> Resistor_SMD:R_0402_1005Metric; LCSC (none) -> C25744
- R67: renamed from R62; footprint (none) -> Resistor_SMD:R_0402_1005Metric; LCSC (none) -> C25744
- R68: renamed from R63; footprint (none) -> Resistor_SMD:R_1206_3216Metric; LCSC C5126235 -> C305315
- R69: renamed from R66; footprint (none) -> Resistor_SMD:R_1206_3216Metric; LCSC C5126235 -> C305315
- R70: renamed from R69; footprint (none) -> Resistor_SMD:R_1206_3216Metric; LCSC C5126235 -> C305315
- R71: renamed from R72; footprint (none) -> Resistor_SMD:R_1206_3216Metric; LCSC C5126235 -> C305315
- R72: renamed from R75; footprint (none) -> Resistor_SMD:R_1206_3216Metric; LCSC C5126235 -> C305315
- R73: renamed from R78; footprint (none) -> Resistor_SMD:R_1206_3216Metric; LCSC C5126235 -> C305315
- R74: renamed from R81; footprint (none) -> Resistor_SMD:R_1206_3216Metric; LCSC C5126235 -> C305315
- R75: renamed from R64; footprint (none) -> Resistor_SMD:R_0402_1005Metric; LCSC (none) -> C11702
- R76: renamed from R67; footprint (none) -> Resistor_SMD:R_0402_1005Metric; LCSC (none) -> C11702
- R77: renamed from R70; footprint (none) -> Resistor_SMD:R_0402_1005Metric; LCSC (none) -> C11702
- R78: renamed from R73; footprint (none) -> Resistor_SMD:R_0402_1005Metric; LCSC (none) -> C11702
- R79: renamed from R76; footprint (none) -> Resistor_SMD:R_0402_1005Metric; LCSC (none) -> C11702
- R80: renamed from R79; footprint (none) -> Resistor_SMD:R_0402_1005Metric; LCSC (none) -> C11702
- R81: renamed from R82; footprint (none) -> Resistor_SMD:R_0402_1005Metric; LCSC (none) -> C11702
- R82: renamed from R65; footprint (none) -> Resistor_SMD:R_0402_1005Metric; LCSC (none) -> C25744
- R83: renamed from R68; footprint (none) -> Resistor_SMD:R_0402_1005Metric; LCSC (none) -> C25744
- R84: renamed from R71; footprint (none) -> Resistor_SMD:R_0402_1005Metric; LCSC (none) -> C25744
- R85: renamed from R74; footprint (none) -> Resistor_SMD:R_0402_1005Metric; LCSC (none) -> C25744
- R86: renamed from R77; footprint (none) -> Resistor_SMD:R_0402_1005Metric; LCSC (none) -> C25744
- R87: renamed from R80; footprint (none) -> Resistor_SMD:R_0402_1005Metric; LCSC (none) -> C25744
- R88: renamed from R83; footprint (none) -> Resistor_SMD:R_0402_1005Metric; LCSC (none) -> C25744
- R89: renamed from R99; footprint (none) -> Resistor_SMD:R_1206_3216Metric; LCSC C5126235 -> C305315
- R90: renamed from R96; footprint (none) -> Resistor_SMD:R_1206_3216Metric; LCSC C5126235 -> C305315
- R91: renamed from R93; footprint (none) -> Resistor_SMD:R_1206_3216Metric; LCSC C5126235 -> C305315
- R92: renamed from R90; footprint (none) -> Resistor_SMD:R_1206_3216Metric; LCSC C5126235 -> C305315
- R93: renamed from R87; footprint (none) -> Resistor_SMD:R_1206_3216Metric; LCSC C5126235 -> C305315
- R94: renamed from R84; footprint (none) -> Resistor_SMD:R_1206_3216Metric; LCSC C5126235 -> C305315
- R95: renamed from R100; footprint (none) -> Resistor_SMD:R_0402_1005Metric; LCSC (none) -> C11702
- R96: renamed from R97; footprint (none) -> Resistor_SMD:R_0402_1005Metric; LCSC (none) -> C11702
- R97: renamed from R94; footprint (none) -> Resistor_SMD:R_0402_1005Metric; LCSC (none) -> C11702
- R98: renamed from R91; footprint (none) -> Resistor_SMD:R_0402_1005Metric; LCSC (none) -> C11702
- R99: renamed from R88; footprint (none) -> Resistor_SMD:R_0402_1005Metric; LCSC (none) -> C11702
- U10: renamed from U15; footprint (none) -> Ultra_librarian:VFQFPN16_STSPIN_STM; LCSC (none) -> C155561
- U11: renamed from U30; footprint (none) -> Ultra_librarian:VFQFPN16_STSPIN_STM; LCSC (none) -> C155561
- U12: renamed from U7; footprint (none) -> Ultra_librarian:VFQFPN16_STSPIN_STM; LCSC (none) -> C155561
- U13: renamed from U2; footprint (none) -> Ultra_librarian:VFQFPN16_STSPIN_STM; LCSC (none) -> C155561
- U14: renamed from U8; footprint (none) -> Ultra_librarian:VFQFPN16_STSPIN_STM; LCSC (none) -> C155561
- U15: renamed from U13; footprint (none) -> Ultra_librarian:VFQFPN16_STSPIN_STM; LCSC (none) -> C155561
- U16: renamed from U12; footprint (none) -> Ultra_librarian:VFQFPN16_STSPIN_STM; LCSC (none) -> C155561
- U17: renamed from U22; footprint (none) -> Ultra_librarian:VFQFPN16_STSPIN_STM; LCSC (none) -> C155561
- U18: renamed from U23; footprint (none) -> Ultra_librarian:VFQFPN16_STSPIN_STM; LCSC (none) -> C155561
- U19: renamed from U32; footprint (none) -> Ultra_librarian:VFQFPN16_STSPIN_STM; LCSC (none) -> C155561
- U20: renamed from U9; footprint (none) -> Ultra_librarian:VFQFPN16_STSPIN_STM; LCSC (none) -> C155561
- U21: renamed from U31; footprint (none) -> Ultra_librarian:VFQFPN16_STSPIN_STM; LCSC (none) -> C155561
- U22: renamed from U16; footprint (none) -> Ultra_librarian:VFQFPN16_STSPIN_STM; LCSC (none) -> C155561
- U23: renamed from U17; footprint (none) -> Ultra_librarian:VFQFPN16_STSPIN_STM; LCSC (none) -> C155561
- U24: renamed from U18; footprint (none) -> Ultra_librarian:VFQFPN16_STSPIN_STM; LCSC (none) -> C155561
- U25: renamed from U19; footprint (none) -> Ultra_librarian:VFQFPN16_STSPIN_STM; LCSC (none) -> C155561
- U26: renamed from U20; footprint (none) -> Ultra_librarian:VFQFPN16_STSPIN_STM; LCSC (none) -> C155561
- U27: renamed from U21; footprint (none) -> Ultra_librarian:VFQFPN16_STSPIN_STM; LCSC (none) -> C155561
- U28: renamed from U33; footprint (none) -> Ultra_librarian:VFQFPN16_STSPIN_STM; LCSC (none) -> C155561
- U29: renamed from U24; footprint (none) -> Ultra_librarian:VFQFPN16_STSPIN_STM; LCSC (none) -> C155561
- U30: renamed from U25; footprint (none) -> Ultra_librarian:VFQFPN16_STSPIN_STM; LCSC (none) -> C155561
- U31: renamed from U26; footprint (none) -> Ultra_librarian:VFQFPN16_STSPIN_STM; LCSC (none) -> C155561
- U32: renamed from U27; footprint (none) -> Ultra_librarian:VFQFPN16_STSPIN_STM; LCSC (none) -> C155561
- U33: renamed from U28; footprint (none) -> Ultra_librarian:VFQFPN16_STSPIN_STM; LCSC (none) -> C155561
- U7: renamed from U11; footprint (none) -> Ultra_librarian:VFQFPN16_STSPIN_STM; LCSC (none) -> C155561
- U8: renamed from U10; footprint (none) -> Ultra_librarian:VFQFPN16_STSPIN_STM; LCSC (none) -> C155561
- U9: renamed from U14; footprint (none) -> Ultra_librarian:VFQFPN16_STSPIN_STM; LCSC (none) -> C155561
- renumbered J8 to J10, J9 to J11, J10 to J12, J5 to J13, J2 to J14, J16 to J15, J15 to J16, J14 to J17, J13 to J18, J12 to J19, J11 to J20, J17 to J21, J18 to J22, J19 to J23, J20 to J24, J21 to J25, J22 to J26, J23 to J27, J24 to J28, J30 to J29, J29 to J30, J28 to J31, J27 to J32, J26 to J33, J25 to J34, J6 to J8, J7 to J9
Connections:
- net +1V8: now also C19.1, C19.1, C19.1, C19.1, C19.1, C19.1, C19.1, C19.1, C19.1, C19.1, C19.1, C19.1, C19.1, C19.1, C19.1, C19.1, C19.1, C19.1, C19.1, C19.1, C19.1, C19.1, C19.1, C19.1, C19.1, C19.1, C19.1
- net DRIVER_ENABLE: now also C19.1
- net GND: now also C19.2, C19.2, C19.2, C19.2, C19.2, C19.2, C19.2, C19.2, C19.2, C19.2, C19.2, C19.2, C19.2, C19.2, C19.2, C19.2, C19.2, C19.2, C19.2, C19.2, C19.2, C19.2, C19.2, C19.2, C19.2, C19.2, C19.2, C19.2
Other:
- moved on the sheet: C38, C46, C47, C48, C49, C50, C51, C52, C60, C61, C62, C63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

Commit message: Add files via upload
Parts:
- removed C19 (x27): 100nF, Capacitor_SMD:C_0402_1005Metric, symbol Device:C_Small
- removed C46, C47, C48, C49, C50, C51, C52, C60, C61, C62, C63, C64, C65, C66, C74, C75, C76, C77, C78, C79, C80, C87, C88, C89, C90, C91, C92: 22nF, Capacitor_SMD:C_0402_1005Metric, symbol Device:C_Small
- removed J10, J11, J12, J13, J14, J15, J16, J17, J18, J19, J20, J21, J22, J23, J24, J25, J26, J27, J28, J29, J30, J31, J32, J33, J34, J8, J9: Picoblade, Connector_Molex:Molex_PicoBlade_53047-0210_1x02_P1.25mm_Vertical, symbol Connector_Generic:Conn_01x02
- removed R100, R33, R34, R35, R36, R37, R38, R39, R54, R55, R56, R57, R58, R59, R60, R75, R76, R77, R78, R79, R80, R81, R95, R96, R97, R98, R99: 1k, Resistor_SMD:R_0402_1005Metric, symbol Device:R_Small_US
- removed R101, R102, R103, R104, R105, R106, R40, R41, R42, R43, R44, R45, R46, R61, R62, R63, R64, R65, R66, R67, R82, R83, R84, R85, R86, R87, R88: 10k, Resistor_SMD:R_0402_1005Metric, symbol Device:R_Small_US
- removed R26, R27, R28, R29, R30, R31, R32, R47, R48, R49, R50, R51, R52, R53, R68, R69, R70, R71, R72, R73, R74, R89, R90, R91, R92, R93, R94: 1.4R, Resistor_SMD:R_1206_3216Metric, symbol Device:R_Small_US
- removed U10, U11, U12, U13, U14, U15, U16, U17, U18, U19, U20, U21, U22, U23, U24, U25, U26, U27, U28, U29, U30, U31, U32, U33, U7, U8, U9: STSPIN250, Ultra_librarian:VFQFPN16_STSPIN_STM, symbol components_2:STSPIN250
Other:
- added sheet HRTIM_CHA1 (HRTIM_CHA1.kicad_sch)
- added sheet HRTIM_CHA2 (HRTIM_CHA2.kicad_sch)
- added sheet HRTIM_CHB1 (HRTIM_CHB1.kicad_sch)
- added sheet HRTIM_CHB2 (HRTIM_CHB2.kicad_sch)
- added sheet HRTIM_CHC1 (HRTIM_CHC1.kicad_sch)
- added sheet HRTIM_CHC2 (HRTIM_CHC2.kicad_sch)
- added sheet HRTIM_CHD1 (HRTIM_CHD1.kicad_sch)
- added sheet HRTIM_CHD2 (HRTIM_CHD2.kicad_sch)
- added sheet LPTIM1_OUT (LPTIM1_OUT.kicad_sch)
- added sheet TIM12_CH2 (TIM12_CH2.kicad_sch)
- added sheet TIM13_CH1 (TIM13_CH1.kicad_sch)
- added sheet TIM14_CH1 (TIM14_CH1.kicad_sch)
- added sheet TIM15_CH1 (TIM15_CH1.kicad_sch)
- added sheet TIM15_CH2 (TIM15_CH2.kicad_sch)
- added sheet TIM16_CH1 (TIM16_CH1.kicad_sch)
- added sheet TIM1_CH1 (TIM1_CH1.kicad_sch)
- added sheet TIM1_CH2 (TIM1_CH2.kicad_sch)
- added sheet TIM1_CH3 (TIM1_CH3.kicad_sch)
- added sheet TIM1_CH4 (TIM1_CH4.kicad_sch)
- added sheet TIM2_CH1 (TIM2_CH1.kicad_sch)
- added sheet TIM4_CH1 (TIM4_CH1.kicad_sch)
- added sheet TIM4_CH2 (TIM4_CH2.kicad_sch)
- added sheet TIM4_CH3 (TIM4_CH3.kicad_sch)
- added sheet TIM4_CH4 (TIM4_CH4.kicad_sch)
- added sheet TIM5_CH2 (TIM5_CH2.kicad_sch)
- added sheet TIM5_CH3 (TIM5_CH3.kicad_sch)
- added sheet TIM8_CH4 (TIM8_CH4.kicad_sch)

Commit message: Add files via upload
Changed lines of the file:
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@@
     (stroke (width 0) (type default))
   )
-  (wire (pts (xy 33.02 38.1) (xy 35.56 38.1))
+  (wire (pts (xy 33.02 38.1) (xy 40.64 38.1))
     (stroke (width 0) (type default))
   )
@@
     (effects (font (size 5 5)) (justify left bottom))
   )
-  (label "EN" (at 71.12 36.83 180) (fields_autoplaced)
-    (effects (font (size 1.27 1.27)) (justify right bottom))
-  )
-  (label "REF" (at 35.56 38.1 0) (fields_autoplaced)
-    (effects (font (size 1.27 1.27)) (justify left bottom))
-  )
   (global_label "DRIVER_ENABLE" (shape input) (at 77.47 36.83 0) (fields_autoplaced)
     (effects (font (size 1.27 1.27)) (justify left))
@@
       (effects (font (size 1.27 1.27)) (justify left) hide)
     )
+  )
+  (global_label "REF" (shape input) (at 40.64 38.1 0) (fields_autoplaced)
+    (effects (font (size 1.27 1.27)) (justify left))
+    (property "Intersheetrefs" "${INTERSHEET_REFS}" (at 47.1328 38.1 0)
+      (effects (font (size 1.27 1.27)) (justify left) hide)
+    )

Commit message: Add files via upload
Parts:
- removed C19: 100nF, Capacitor_SMD:C_0402_1005Metric, symbol Device:C_Small
- removed R23: 10k, Resistor_SMD:R_0402_1005Metric, symbol Device:R_Small_US
Other:
- note removed: "EN is MCU Open-Drain Output (PA15)"
Changed lines of the file:
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@@
   (junction (at 27.94 38.1) (diameter 0) (color 0 0 0 0)
-  )
-  (junction (at 66.04 36.83) (diameter 0) (color 0 0 0 0)
   )
   (junction (at 27.94 44.45) (diameter 0) (color 0 0 0 0)
@@
   )
   (wire (pts (xy 27.94 44.45) (xy 27.94 45.72))
-    (stroke (width 0) (type default))
-  )
-  (wire (pts (xy 66.04 43.18) (xy 66.04 44.45))
     (stroke (width 0) (type default))
   )
@@
     (stroke (width 0) (type default))
   )
-  (wire (pts (xy 66.04 36.83) (xy 77.47 36.83))
-    (stroke (width 0) (type default))
-  )
-  (wire (pts (xy 66.04 35.56) (xy 66.04 36.83))
-    (stroke (width 0) (type default))
-  )
   (wire (pts (xy 27.94 31.75) (xy 27.94 33.02))
-    (stroke (width 0) (type default))
-  )
-  (wire (pts (xy 66.04 36.83) (xy 66.04 38.1))
     (stroke (width 0) (type default))
   )
@@
     (stroke (width 0) (type default))
   )
-  (text "EN is MCU Open-Drain Output (PA15)" (at 69.215 33.655 0)
-    (effects (font (size 1.27 1.27)) (justify left bottom))
-  )
   (text "VREF = 0.5V" (at 33.655 34.29 0)
     (effects (font (size 1.27 1.27)) (justify left bottom))
@@
     (at 85.725 24.13 0)
     (effects (font (size 5 5)) (justify left bottom))
-  )
-  (global_label "DRIVER_ENABLE" (shape input) (at 77.47 36.83 0) (fields_autoplaced)
-    (effects (font (size 1.27 1.27)) (justify left))
-    (property "Intersheetrefs" "${INTERSHEET_REFS}" (at 95.0904 36.83 0)
-      (effects (font (size 1.27 1.27)) (justify left) hide)
-    )
   )
   (global_label "REF" (shape input) (at 40.64 38.1 0) (fields_autoplaced)
@@
     )
   )
-  (symbol (lib_id "power:+1V8") (at 66.04 30.48 0) (unit 1)
-    (in_bom yes) (on_board yes) (dnp no)
-    (property "Reference" "#PWR030" (at 66.04 34.29 0)
-      (effects (font (size 1.27 1.27)) hide)
-    )
-    (property "Value" "+1V8" (at 62.865 27.94 0)
-      (effects (font (size 1.27 1.27)))
-    )
-    (property "Footprint" "" (at 66.04 30.48 0)
-      (effects (font (size 1.27 1.27)) hide)
-    )
-    (property "Datasheet" "" (at 66.04 30.48 0)
-      (effects (font (size 1.27 1.27)) hide)
-    )
-    (pin "1")
-    (instances
-      (project "KASM_PCB_REV1"
-        (path "/bcd76057-59fd-41c5-bb52-9bafb2ef74e0/9f28d78d-ca42-4041-9be6-b996c46b4a0a"
-          (reference "#PWR030") (unit 1)
-        )
-        (path "/bcd76057-59fd-41c5-bb52-9bafb2ef74e0/04e958db-aa3d-41e7-905b-1283accbf3a5"
-          (reference "#PWR062") (unit 1)
-        )
-      )
-    )
-  )
-  (symbol (lib_id "Device:R_Small_US") (at 66.04 33.02 0) (unit 1)
-    (in_bom yes) (on_board yes) (dnp no)
-    (property "Reference" "R23" (at 64.135 34.925 0)
-      (effects (font (size 1.27 1.27)) (justify right))
-    )
-    (property "Value" "10k" (at 64.77 32.385 0)
-      (effects (font (size 1.27 1.27)) (justify right))
-    )
-    (property "Footprint" "Resistor_SMD:R_0402_1005Metric" (at 66.04 33.02 0)
-      (effects (font (size 1.27 1.27)) hide)
-    )
-    (property "Datasheet" "~" (at 66.04 33.02 0)
-      (effects (font (size 1.27 1.27)) hide)
-    )
-    (property "LCSC" "C25744" (at 66.04 33.02 0)
-      (effects (font (size 1.27 1.27)) hide)
-    )
-    (pin "1")
-    (pin "2")
-    (instances
-      (project "KASM_PCB_REV1"
-        (path "/bcd76057-59fd-41c5-bb52-9bafb2ef74e0/04e958db-aa3d-41e7-905b-1283accbf3a5"
-          (reference "R23") (unit 1)
-        )
-      )
-    )
-  )
-  (symbol (lib_id "Device:C_Small") (at 66.04 40.64 0) (mirror y) (unit 1)
-    (in_bom yes) (on_board yes) (dnp no)
-    (property "Reference" "C19" (at 63.7159 39.4342 0)
-      (effects (font (size 1.27 1.27)) (justify left))
-    )
-    (property "Value" "100nF" (at 63.7159 41.8584 0)
-      (effects (font (size 1.27 1.27)) (justify left))
-    )
-    (property "Footprint" "Capacitor_SMD:C_0402_1005Metric" (at 66.04 40.64 0)
-      (effects (font (size 1.27 1.27)) hide)
-    )
-    (property "Datasheet" "~" (at 66.04 40.64 0)
-      (effects (font (size 1.27 1.27)) hide)
-    )
-    (property "LCSC" "C1525" (at 66.04 40.64 0)
-      (effects (font (size 1.27 1.27)) hide)
-    )
-    (pin "1")
-    (pin "2")
-    (instances
-      (project "KASM_PCB_REV1"
-        (path "/bcd76057-59fd-41c5-bb52-9bafb2ef74e0/9f28d78d-ca42-4041-9be6-b996c46b4a0a"
-          (reference "C19") (unit 1)
-        )
-        (path "/bcd76057-59fd-41c5-bb52-9bafb2ef74e0/da6e1dd6-6549-4588-8765-3ff657cbe17b"
-          (reference "C1") (unit 1)
-        )
-        (path "/bcd76057-59fd-41c5-bb52-9bafb2ef74e0/04e958db-aa3d-41e7-905b-1283accbf3a5"
-          (reference "C37") (unit 1)
-        )
-      )
-    )
-  )
   (symbol (lib_id "power:GND") (at 27.94 45.72 0) (unit 1)
     (in_bom yes) (on_board yes) (dnp no)
@@
         )
       )
-    )
-  )
-  (symbol (lib_id "power:GND") (at 66.04 44.45 0) (unit 1)
-    (in_bom yes) (on_board yes) (dnp no)
-    (property "Reference" "#PWR064" (at 66.04 50.8 0)
-      (effects (font (size 1.27 1.27)) hide)
-    )
-    (property "Value" "GND" (at 66.04 48.5831 0)
-      (effects (font (size 1.27 1.27)))
-    )
-    (property "Footprint" "" (at 66.04 44.45 0)
-      (effects (font (size 1.27 1.27)) hide)
-    )
-    (property "Datasheet" "" (at 66.04 44.45 0)
-      (effects (font (size 1.27 1.27)) hide)
-    )
-    (pin "1")
-    (instances
-      (project "KASM_PCB_REV1"
-        (path "/bcd76057-59fd-41c5-bb52-9bafb2ef74e0/04e958db-aa3d-41e7-905b-1283accbf3a5"
-          (reference "#PWR064") (unit 1)
-        )
-      )
