File: HRTIM_CHB1.kicad_sch (KiCad schematic)
At the start: 7 parts, among them J13 Picoblade, U12 STSPIN250

Commit message: Add files via upload
Changed lines of the file:
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@@
     (stroke (width 0) (type default))
-  )
-  (label "REF" (at 118.11 102.87 0) (fields_autoplaced)
-    (effects (font (size 1.27 1.27)) (justify left bottom))
   )
   (label "EN" (at 120.65 90.17 0) (fields_autoplaced)
@@
       (effects (font (size 1.27 1.27)) (justify right) hide)
     )
+  )
+  (global_label "REF" (shape input) (at 118.11 102.87 180) (fields_autoplaced)
+    (effects (font (size 1.27 1.27)) (justify right))
+    (property "Intersheetrefs" "${INTERSHEET_REFS}" (at 111.6172 102.87 0)
+      (effects (font (size 1.27 1.27)) (justify right) hide)
+    )

Commit message: Add files via upload
Parts:
- added C19: 100nF, Capacitor_SMD:C_0402_1005Metric, symbol Device:C_Small
- added R23: 10k, Resistor_SMD:R_0402_1005Metric, symbol Device:R_Small_US
Connections:
- net +1V8: now also R23.1
- net EN: now also C19.1, R23.2
- net GND: now also C19.2
Changed lines of the file:
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@@
   (junction (at 156.21 100.33) (diameter 0) (color 0 0 0 0)
   )
+  (junction (at 76.2 63.5) (diameter 0) (color 0 0 0 0)
+  )
   (junction (at 143.51 111.76) (diameter 0) (color 0 0 0 0)
   )
@@
     (stroke (width 0) (type default))
   )
+  (wire (pts (xy 76.2 69.85) (xy 76.2 71.12))
+    (stroke (width 0) (type default))
+  )
   (wire (pts (xy 143.51 111.76) (xy 143.51 110.49))
     (stroke (width 0) (type default))
   )
+  (wire (pts (xy 76.2 62.23) (xy 76.2 63.5))
+    (stroke (width 0) (type default))
+  )
   (wire (pts (xy 156.21 100.33) (xy 156.21 104.14))
     (stroke (width 0) (type default))
@@
     (stroke (width 0) (type default))
   )
+  (wire (pts (xy 76.2 63.5) (xy 82.55 63.5))
+    (stroke (width 0) (type default))
+  )
   (wire (pts (xy 156.21 85.09) (xy 158.75 85.09))
     (stroke (width 0) (type default))
@@
     (stroke (width 0) (type default))
   )
+  (wire (pts (xy 76.2 63.5) (xy 76.2 64.77))
+    (stroke (width 0) (type default))
+  )
   (wire (pts (xy 152.4 82.55) (xy 156.21 82.55))
     (stroke (width 0) (type default))
@@
   (wire (pts (xy 152.4 80.01) (xy 156.21 80.01))
     (stroke (width 0) (type default))
+  )
+  (label "EN" (at 82.55 63.5 180) (fields_autoplaced)
+    (effects (font (size 1.27 1.27)) (justify right bottom))
   )
   (label "EN" (at 120.65 90.17 0) (fields_autoplaced)
@@
     (property "Intersheetrefs" "${INTERSHEET_REFS}" (at 111.6172 102.87 0)
       (effects (font (size 1.27 1.27)) (justify right) hide)
+    )
+  )
+  (symbol (lib_id "Device:R_Small_US") (at 76.2 59.69 0) (unit 1)
+    (in_bom yes) (on_board yes) (dnp no)
+    (property "Reference" "R23" (at 74.295 61.595 0)
+      (effects (font (size 1.27 1.27)) (justify right))
+    )
+    (property "Value" "10k" (at 74.93 59.055 0)
+      (effects (font (size 1.27 1.27)) (justify right))
+    )
+    (property "Footprint" "Resistor_SMD:R_0402_1005Metric" (at 76.2 59.69 0)
+      (effects (font (size 1.27 1.27)) hide)
+    )
+    (property "Datasheet" "~" (at 76.2 59.69 0)
+      (effects (font (size 1.27 1.27)) hide)
+    )
+    (property "LCSC" "C25744" (at 76.2 59.69 0)
+      (effects (font (size 1.27 1.27)) hide)
+    )
+    (pin "1")
+    (pin "2")
+    (instances
+      (project "KASM_PCB_REV1"
+        (path "/bcd76057-59fd-41c5-bb52-9bafb2ef74e0/04e958db-aa3d-41e7-905b-1283accbf3a5"
+          (reference "R23") (unit 1)
+        )
+        (path "/bcd76057-59fd-41c5-bb52-9bafb2ef74e0/04e958db-aa3d-41e7-905b-1283accbf3a5/317da025-5f62-4c93-8d06-7954e608af1c"
+          (reference "R23") (unit 1)
+        )
+        (path "/bcd76057-59fd-41c5-bb52-9bafb2ef74e0/04e958db-aa3d-41e7-905b-1283accbf3a5/18dc00ae-3159-4780-b672-12977f79e5ac"
+          (reference "R57") (unit 1)
+        )
+      )
     )
   )
@@
     )
   )
+  (symbol (lib_id "power:GND") (at 76.2 71.12 0) (unit 1)
+    (in_bom yes) (on_board yes) (dnp no)
+    (property "Reference" "#PWR064" (at 76.2 77.47 0)
+      (effects (font (size 1.27 1.27)) hide)
+    )
+    (property "Value" "GND" (at 76.2 75.2531 0)
+      (effects (font (size 1.27 1.27)))
+    )
+    (property "Footprint" "" (at 76.2 71.12 0)
+      (effects (font (size 1.27 1.27)) hide)
+    )
+    (property "Datasheet" "" (at 76.2 71.12 0)
+      (effects (font (size 1.27 1.27)) hide)
+    )
+    (pin "1")
+    (instances
+      (project "KASM_PCB_REV1"
+        (path "/bcd76057-59fd-41c5-bb52-9bafb2ef74e0/04e958db-aa3d-41e7-905b-1283accbf3a5"
+          (reference "#PWR064") (unit 1)
+        )
+        (path "/bcd76057-59fd-41c5-bb52-9bafb2ef74e0/04e958db-aa3d-41e7-905b-1283accbf3a5/317da025-5f62-4c93-8d06-7954e608af1c"
+          (reference "#PWR015") (unit 1)
+        )
+        (path "/bcd76057-59fd-41c5-bb52-9bafb2ef74e0/04e958db-aa3d-41e7-905b-1283accbf3a5/18dc00ae-3159-4780-b672-12977f79e5ac"
+          (reference "#PWR0132") (unit 1)
+        )
+      )
+    )
+  )
   (symbol (lib_id "Device:R_Small_US") (at 156.21 106.68 0) (mirror y) (unit 1)
     (in_bom yes) (on_board yes) (dnp no)
@@
         )
       )
+    )
+  )
+  (symbol (lib_id "power:+1V8") (at 76.2 57.15 0) (unit 1)
+    (in_bom yes) (on_board yes) (dnp no)
+    (property "Reference" "#PWR030" (at 76.2 60.96 0)
+      (effects (font (size 1.27 1.27)) hide)
+    )
+    (property "Value" "+1V8" (at 73.025 54.61 0)
+      (effects (font (size 1.27 1.27)))
+    )
+    (property "Footprint" "" (at 76.2 57.15 0)
+      (effects (font (size 1.27 1.27)) hide)
+    )
+    (property "Datasheet" "" (at 76.2 57.15 0)
+      (effects (font (size 1.27 1.27)) hide)
+    )
+    (pin "1")
+    (instances
+      (project "KASM_PCB_REV1"
+        (path "/bcd76057-59fd-41c5-bb52-9bafb2ef74e0/9f28d78d-ca42-4041-9be6-b996c46b4a0a"
+          (reference "#PWR030") (unit 1)
+        )
+        (path "/bcd76057-59fd-41c5-bb52-9bafb2ef74e0/04e958db-aa3d-41e7-905b-1283accbf3a5"
+          (reference "#PWR062") (unit 1)
+        )
+        (path "/bcd76057-59fd-41c5-bb52-9bafb2ef74e0/04e958db-aa3d-41e7-905b-1283accbf3a5/317da025-5f62-4c93-8d06-7954e608af1c"
+          (reference "#PWR014") (unit 1)
+        )
+        (path "/bcd76057-59fd-41c5-bb52-9bafb2ef74e0/04e958db-aa3d-41e7-905b-1283accbf3a5/18dc00ae-3159-4780-b672-12977f79e5ac"
+          (reference "#PWR0131") (unit 1)
+        )
+      )
+    )
+  )
+  (symbol (lib_id "Device:C_Small") (at 76.2 67.31 0) (mirror y) (unit 1)
+    (in_bom yes) (on_board yes) (dnp no)
+    (property "Reference" "C19" (at 73.8759 66.1042 0)
+      (effects (font (size 1.27 1.27)) (justify left))
+    )
+    (property "Value" "100nF" (at 73.8759 68.5284 0)
+      (effects (font (size 1.27 1.27)) (justify left))
+    )
+    (property "Footprint" "Capacitor_SMD:C_0402_1005Metric" (at 76.2 67.31 0)
+      (effects (font (size 1.27 1.27)) hide)
+    )
+    (property "Datasheet" "~" (at 76.2 67.31 0)
+      (effects (font (size 1.27 1.27)) hide)
+    )
+    (property "LCSC" "C1525" (at 76.2 67.31 0)
+      (effects (font (size 1.27 1.27)) hide)
+    )
+    (pin "1")
+    (pin "2")
+    (instances
+      (project "KASM_PCB_REV1"
+        (path "/bcd76057-59fd-41c5-bb52-9bafb2ef74e0/9f28d78d-ca42-4041-9be6-b996c46b4a0a"
+          (reference "C19") (unit 1)
+        )
+        (path "/bcd76057-59fd-41c5-bb52-9bafb2ef74e0/da6e1dd6-6549-4588-8765-3ff657cbe17b"
+          (reference "C1") (unit 1)
+        )
+        (path "/bcd76057-59fd-41c5-bb52-9bafb2ef74e0/04e958db-aa3d-41e7-905b-1283accbf3a5"
+          (reference "C37") (unit 1)
+        )
+        (path "/bcd76057-59fd-41c5-bb52-9bafb2ef74e0/04e958db-aa3d-41e7-905b-1283accbf3a5/317da025-5f62-4c93-8d06-7954e608af1c"
+          (reference "C37") (unit 1)
+        )
+        (path "/bcd76057-59fd-41c5-bb52-9bafb2ef74e0/04e958db-aa3d-41e7-905b-1283accbf3a5/18dc00ae-3159-4780-b672-12977f79e5ac"
+          (reference "C72") (unit 1)
+        )
+      )

Commit message: Add files via upload
Parts:
- C19: value 100nF -> 10nF; LCSC C1525 -> C15195
- R31: value 1.4R -> 1.0R; LCSC C305315 -> C17928
Changed lines of the file:
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@@
       (effects (font (size 1.27 1.27)) (justify right))
     )
-    (property "Value" "1.4R" (at 157.861 107.8921 0)
+    (property "Value" "1.0R" (at 157.861 107.8921 0)
       (effects (font (size 1.27 1.27)) (justify right))
     )
@@
       (effects (font (size 1.27 1.27)) hide)
     )
-    (property "LCSC" "C305315" (at 156.21 106.68 0)
+    (property "LCSC" "C17928" (at 156.21 106.68 0)
       (effects (font (size 1.27 1.27)) hide)
     )
@@
       (effects (font (size 1.27 1.27)) (justify left))
     )
-    (property "Value" "100nF" (at 73.8759 68.5284 0)
+    (property "Value" "10nF" (at 73.8759 68.5284 0)
       (effects (font (size 1.27 1.27)) (justify left))
     )
@@
       (effects (font (size 1.27 1.27)) hide)
     )
-    (property "LCSC" "C1525" (at 76.2 67.31 0)
-      (effects (font (size 1.27 1.27)) hide)
-    )
+    (property "LCSC" "C15195" (at 76.2 67.31 0)
+      (effects (font (size 1.27 1.27)) hide)
+    )
