File: KASM_PCB_REV1_POWER.kicad_sch (KiCad schematic)
At the start: 40 parts, among them J34 Conn_01x02, J4 Barrel_Jack_Switch, U3 TPS5430DDA, U4 TPS54620

Commit message: Add files via upload
Parts:
- C5: renamed from C14; footprint (none) -> Capacitor_SMD:C_0402_1005Metric; LCSC (none) -> C1525
- C6: renamed from C16; footprint (none) -> Capacitor_SMD:CP_Elec_6.3x5.4
- C7: renamed from C27; footprint (none) -> Capacitor_SMD:CP_Elec_6.3x5.4
- J2: renamed from J34; value Conn_01x02 -> Screw Terminal; LCSC (none) -> C557646
- renumbered C15 to C1, C29 to C10, C22 to C11, C19 to C12, C31 to C13, C30 to C14, C32 to C15, C33 to C16, C21 to C17, C25 to C18, C24 to C19, C13 to C2, C23 to C20, C17 to C3, C18 to C4, C20 to C8, C28 to C9, D3 to D2, D2 to D3, J4 to J1, L2 to L1, L3 to L2, R2 to R1, R9 to R10, R4 to R2, R5 to R4, R6 to R5, R10 to R6, R12 to R9, U3 to U1, U4 to U2
Other:
- note added: "12V CONNECTORS"
- moved on the sheet: C1, C10, C11, C12, C13, C14, C15, C16, C17, C18, C19, C2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

Commit message: Add files via upload
Parts:
- removed D3: D_Schottky, Diode_SMD:D_SMA, symbol Device:D_Schottky
- added C93: 100nF, Capacitor_SMD:C_0402_1005Metric, symbol Device:C
- D1: footprint Diode_SMD:D_SMA -> Diode_SMD:D_SOD-323; LCSC C8678 -> C191023
Connections:
- net +12V: now also C93.1
- net GND: now also C93.2
Other:
- moved on the sheet: C10, C11, C8, C9

Commit message: Add files via upload
Parts:
- added C39, C44: 100nF, Capacitor_SMD:C_0402_1005Metric, symbol Device:C_Small
- added C9 (x2): 4.7uF, Capacitor_SMD:C_0402_1005Metric, symbol Device:C_Small
- added FB1, FB2: FerriteBead_Small, Inductor_SMD:L_0805_2012Metric, symbol Device:FerriteBead_Small
- added H1, H2, H3, H4: MountingHole_Pad, MountingHole:MountingHole_3.2mm_M3_DIN965_Pad, symbol Mechanical:MountingHole_Pad
Connections:
- net +12V: now also C39.1, C44.1, C9.2, C9.2, FB1.1, FB2.1; no longer C10.1, C11.1, C2.1, C3.1, C4.1, C5.1, C8.1, C9.1, C93.1, D2.2 (A), R1.1, R5.1, U1.7 (VIN), U2.4 (PVIN), U2.5 (PVIN), U2.6 (VIN)
- net GND: now also C39.2, C44.2, C9.1, C9.1, H1.1, H2.1, H3.1, H4.1
- net +3V3 renamed +3.3V
- new net: C10.1, C11.1, C8.1, C9.1, C93.1, D2.2 (A), FB2.2, R5.1, U2.4 (PVIN), U2.5 (PVIN), U2.6 (VIN)
- new net: C2.1, C3.1, C4.1, C5.1, FB1.2, R1.1, U1.7 (VIN)
Other:
- note added: "MOUNTING HOLES"

Commit message: Add files via upload
Changed lines of the file:
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@@
-    (stroke (width 0) (type default))
-  )
-  (wire (pts (xy 60.96 245.11) (xy 63.5 245.11))
     (stroke (width 0) (type default))
   )
@@
     (stroke (width 0) (type default))
   )
-  (wire (pts (xy 60.96 246.38) (xy 60.96 245.11))
-    (stroke (width 0) (type default))
-  )
   (wire (pts (xy 217.17 73.66) (xy 217.17 74.93))
     (stroke (width 0) (type default))
@@
   )
   (wire (pts (xy 236.22 80.01) (xy 236.22 78.74))
-    (stroke (width 0) (type default))
-  )
-  (wire (pts (xy 54.61 246.38) (xy 60.96 246.38))
     (stroke (width 0) (type default))
   )
@@
     )
   )
-  (symbol (lib_id "power:GND") (at 63.5 245.11 0) (unit 1)
-    (in_bom yes) (on_board yes) (dnp no) (fields_autoplaced)
-    (property "Reference" "#PWR066" (at 63.5 251.46 0)
-      (effects (font (size 1.27 1.27)) hide)
-    )
-    (property "Value" "GND" (at 63.5 249.2431 0)
-      (effects (font (size 1.27 1.27)))
-    )
-    (property "Footprint" "" (at 63.5 245.11 0)
-      (effects (font (size 1.27 1.27)) hide)
-    )
-    (property "Datasheet" "" (at 63.5 245.11 0)
-      (effects (font (size 1.27 1.27)) hide)
-    )
+  (symbol (lib_id "power:GND") (at 54.61 246.38 0) (unit 1)
+    (in_bom yes) (on_board yes) (dnp no) (fields_autoplaced)
+    (property "Reference" "#PWR066" (at 54.61 252.73 0)
+      (effects (font (size 1.27 1.27)) hide)
+    )
+    (property "Value" "GND" (at 54.61 250.5131 0)
+      (effects (font (size 1.27 1.27)))
+    )
+    (property "Footprint" "" (at 54.61 246.38 0)
+      (effects (font (size 1.27 1.27)) hide)
+    )
+    (property "Datasheet" "" (at 54.61 246.38 0)
+      (effects (font (size 1.27 1.27)) hide)
+    )

Commit message: Add files via upload
Parts:
- removed C9 (x2): 4.7uF, Capacitor_SMD:C_0402_1005Metric, symbol Device:C_Small
- added C41, C43: 10uF, Capacitor_SMD:C_1206_3216Metric, symbol Device:C
Connections:
- net +12V: now also C41.1, C43.1
- net GND: now also C41.2, C43.2
Changed lines of the file:
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@@
   (junction (at 251.46 151.13) (diameter 0) (color 0 0 0 0)
   )
+  (junction (at 142.24 63.5) (diameter 0) (color 0 0 0 0)
+  )
   (junction (at 240.03 161.29) (diameter 0) (color 0 0 0 0)
   )
@@
   (junction (at 285.75 68.58) (diameter 0) (color 0 0 0 0)
   )
+  (junction (at 142.24 73.66) (diameter 0) (color 0 0 0 0)
+  )
   (junction (at 304.8 151.13) (diameter 0) (color 0 0 0 0)
   )
@@
   (junction (at 96.52 147.32) (diameter 0) (color 0 0 0 0)
   )
-  (junction (at 142.24 63.5) (diameter 0) (color 0 0 0 0)
-  )
   (junction (at 180.34 63.5) (diameter 0) (color 0 0 0 0)
   )
@@
   )
   (junction (at 242.57 151.13) (diameter 0) (color 0 0 0 0)
-  )
-  (junction (at 142.24 73.66) (diameter 0) (color 0 0 0 0)
   )
   (junction (at 217.17 137.16) (diameter 0) (color 0 0 0 0)
@@
     (stroke (width 0) (type default))
   )
+  (wire (pts (xy 96.52 146.05) (xy 96.52 147.32))
+    (stroke (width 0) (type default))
+  )
   (wire (pts (xy 325.12 151.13) (xy 335.28 151.13))
     (stroke (width 0) (type default))
@@
     (stroke (width 0) (type default))
   )
-  (wire (pts (xy 142.24 71.12) (xy 142.24 73.66))
-    (stroke (width 0) (type default))
-  )
   (wire (pts (xy 220.98 170.18) (xy 224.79 170.18))
     (stroke (width 0) (type default))
@@
     (stroke (width 0) (type default))
   )
-  (wire (pts (xy 142.24 63.5) (xy 142.24 66.04))
-    (stroke (width 0) (type default))
-  )
   (wire (pts (xy 142.24 63.5) (xy 153.67 63.5))
     (stroke (width 0) (type default))
@@
     (stroke (width 0) (type default))
   )
+  (wire (pts (xy 142.24 64.77) (xy 142.24 63.5))
+    (stroke (width 0) (type default))
+  )
   (wire (pts (xy 123.19 147.32) (xy 134.62 147.32))
     (stroke (width 0) (type default))
@@
     (stroke (width 0) (type default))
   )
-  (wire (pts (xy 96.52 144.78) (xy 96.52 147.32))
-    (stroke (width 0) (type default))
-  )
   (wire (pts (xy 248.92 63.5) (xy 254 63.5))
     (stroke (width 0) (type default))
@@
     (stroke (width 0) (type default))
   )
+  (wire (pts (xy 142.24 72.39) (xy 142.24 73.66))
+    (stroke (width 0) (type default))
+  )
   (wire (pts (xy 163.83 63.5) (xy 168.91 63.5))
     (stroke (width 0) (type default))
@@
     (stroke (width 0) (type default))
   )
-  (wire (pts (xy 96.52 137.16) (xy 96.52 139.7))
+  (wire (pts (xy 96.52 137.16) (xy 96.52 138.43))
     (stroke (width 0) (type default))
   )
@@
   (text "MCU POWER" (at 212.09 46.99 0)
     (effects (font (size 5 5)) (justify left bottom))
-  )
-  (symbol (lib_id "Device:C_Small") (at 142.24 68.58 0) (mirror x) (unit 1)
-    (in_bom yes) (on_board yes) (dnp no)
-    (property "Reference" "C9" (at 139.9159 67.3615 0)
-      (effects (font (size 1.27 1.27)) (justify right))
-    )
-    (property "Value" "4.7uF" (at 139.9159 69.7857 0)
-      (effects (font (size 1.27 1.27)) (justify right))
-    )
-    (property "Footprint" "Capacitor_SMD:C_0402_1005Metric" (at 142.24 68.58 0)
-      (effects (font (size 1.27 1.27)) hide)
-    )
-    (property "Datasheet" "~" (at 142.24 68.58 0)
-      (effects (font (size 1.27 1.27)) hide)
-    )
-    (property "LCSC" "C23733" (at 142.24 68.58 0)
-      (effects (font (size 1.27 1.27)) hide)
-    )
-    (pin "1")
-    (pin "2")
-    (instances
-      (project "KASM_PCB_REV1"
-        (path "/bcd76057-59fd-41c5-bb52-9bafb2ef74e0"
-          (reference "C9") (unit 1)
-        )
-        (path "/bcd76057-59fd-41c5-bb52-9bafb2ef74e0/da6e1dd6-6549-4588-8765-3ff657cbe17b"
-          (reference "C27") (unit 1)
-        )
-        (path "/bcd76057-59fd-41c5-bb52-9bafb2ef74e0/9f28d78d-ca42-4041-9be6-b996c46b4a0a"
-          (reference "C41") (unit 1)
-        )
-      )
-    )
   )
   (symbol (lib_id "power:GND") (at 233.68 81.28 0) (unit 1)
@@
         (path "/bcd76057-59fd-41c5-bb52-9bafb2ef74e0/9f28d78d-ca42-4041-9be6-b996c46b4a0a"
           (reference "#PWR027") (unit 1)
-        )
-      )
-    )
-  )
-  (symbol (lib_id "Device:C_Small") (at 96.52 142.24 0) (mirror x) (unit 1)
-    (in_bom yes) (on_board yes) (dnp no)
-    (property "Reference" "C9" (at 94.1959 141.0215 0)
-      (effects (font (size 1.27 1.27)) (justify right))
-    )
-    (property "Value" "4.7uF" (at 94.1959 143.4457 0)
-      (effects (font (size 1.27 1.27)) (justify right))
-    )
-    (property "Footprint" "Capacitor_SMD:C_0402_1005Metric" (at 96.52 142.24 0)
-      (effects (font (size 1.27 1.27)) hide)
-    )
-    (property "Datasheet" "~" (at 96.52 142.24 0)
-      (effects (font (size 1.27 1.27)) hide)
-    )
-    (property "LCSC" "C23733" (at 96.52 142.24 0)
-      (effects (font (size 1.27 1.27)) hide)
-    )
-    (pin "1")
-    (pin "2")
-    (instances
-      (project "KASM_PCB_REV1"
-        (path "/bcd76057-59fd-41c5-bb52-9bafb2ef74e0"
-          (reference "C9") (unit 1)
-        )
-        (path "/bcd76057-59fd-41c5-bb52-9bafb2ef74e0/da6e1dd6-6549-4588-8765-3ff657cbe17b"
-          (reference "C27") (unit 1)
-        )
-        (path "/bcd76057-59fd-41c5-bb52-9bafb2ef74e0/9f28d78d-ca42-4041-9be6-b996c46b4a0a"
-          (reference "C43") (unit 1)
         )
       )
@@
         )
       )
+    )
+  )
+  (symbol (lib_id "Device:C") (at 96.52 142.24 0) (mirror y) (unit 1)
+    (in_bom yes) (on_board yes) (dnp no)
+    (property "Reference" "C43" (at 93.599 141.0279 0)
+      (effects (font (size 1.27 1.27)) (justify left))
+    )
+    (property "Value" "10uF" (at 93.599 143.4521 0)
+      (effects (font (size 1.27 1.27)) (justify left))
+    )
+    (property "Footprint" "Capacitor_SMD:C_1206_3216Metric" (at 95.5548 146.05 0)
+      (effects (font (size 1.27 1.27)) hide)
+    )
+    (property "Datasheet" "~" (at 96.52 142.24 0)
+      (effects (font (size 1.27 1.27)) hide)
+    )
+    (property "LCSC" "C454102" (at 96.52 142.24 0)
+      (effects (font (size 1.27 1.27)) hide)
+    )
+    (pin "1")
+    (pin "2")
+    (instances
+      (project "KASM_PCB_REV1"
+        (path "/bcd76057-59fd-41c5-bb52-9bafb2ef74e0/9f28d78d-ca42-4041-9be6-b996c46b4a0a"
+          (reference "C43") (unit 1)
+        )
+      )
+    )
+  )
+  (symbol (lib_id "Device:C") (at 142.24 68.58 0) (mirror y) (unit 1)
+    (in_bom yes) (on_board yes) (dnp no)
+    (property "Reference" "C41" (at 139.319 67.3679 0)
+      (effects (font (size 1.27 1.27)) (justify left))
+    )
+    (property "Value" "10uF" (at 139.319 69.7921 0)
+      (effects (font (size 1.27 1.27)) (justify left))
+    )
+    (property "Footprint" "Capacitor_SMD:C_1206_3216Metric" (at 141.2748 72.39 0)
+      (effects (font (size 1.27 1.27)) hide)
+    )
+    (property "Datasheet" "~" (at 142.24 68.58 0)
+      (effects (font (size 1.27 1.27)) hide)
+    )
+    (property "LCSC" "C454102" (at 142.24 68.58 0)
+      (effects (font (size 1.27 1.27)) hide)
+    )
+    (pin "1")
+    (pin "2")
+    (instances
+      (project "KASM_PCB_REV1"
+        (path "/bcd76057-59fd-41c5-bb52-9bafb2ef74e0/9f28d78d-ca42-4041-9be6-b996c46b4a0a"
+          (reference "C41") (unit 1)
+        )
+      )
