File: TIM4_CH1.kicad_sch (KiCad schematic)
At the start: 7 parts, among them J13 Picoblade, U12 STSPIN250

Commit message: Add files via upload
Changed lines of the file:
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@@
-    (stroke (width 0) (type default))
-  )
-  (wire (pts (xy 118.11 102.87) (xy 124.46 102.87))
     (stroke (width 0) (type default))
   )
@@
   )
   (wire (pts (xy 119.38 80.01) (xy 124.46 80.01))
+    (stroke (width 0) (type default))
+  )
+  (wire (pts (xy 118.11 102.87) (xy 124.46 102.87))
     (stroke (width 0) (type default))
   )
@@
     (stroke (width 0) (type default))
   )
-  (label "REF" (at 118.11 102.87 0) (fields_autoplaced)
-    (effects (font (size 1.27 1.27)) (justify left bottom))
-  )
   (label "EN" (at 120.65 90.17 0) (fields_autoplaced)
     (effects (font (size 1.27 1.27)) (justify left bottom))
   )
+  (global_label "REF" (shape input) (at 118.11 102.87 180) (fields_autoplaced)
+    (effects (font (size 1.27 1.27)) (justify right))
+    (property "Intersheetrefs" "${INTERSHEET_REFS}" (at 111.6172 102.87 0)
+      (effects (font (size 1.27 1.27)) (justify right) hide)
+    )
+  )
   (global_label "TIM4_CH1" (shape input) (at 119.38 82.55 180) (fields_autoplaced)

Commit message: Add files via upload
Parts:
- added C19: 100nF, Capacitor_SMD:C_0402_1005Metric, symbol Device:C_Small
- added R23: 10k, Resistor_SMD:R_0402_1005Metric, symbol Device:R_Small_US
Connections:
- net +1V8: now also R23.1
- net EN: now also C19.1, R23.2
- net GND: now also C19.2
Changed lines of the file:
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@@
   (junction (at 156.21 100.33) (diameter 0) (color 0 0 0 0)
   )
+  (junction (at 69.85 64.77) (diameter 0) (color 0 0 0 0)
+  )
   (junction (at 143.51 111.76) (diameter 0) (color 0 0 0 0)
   )
@@
     (stroke (width 0) (type default))
   )
+  (wire (pts (xy 69.85 71.12) (xy 69.85 72.39))
+    (stroke (width 0) (type default))
+  )
   (wire (pts (xy 115.57 91.44) (xy 115.57 92.71))
     (stroke (width 0) (type default))
@@
     (stroke (width 0) (type default))
   )
+  (wire (pts (xy 69.85 64.77) (xy 76.2 64.77))
+    (stroke (width 0) (type default))
+  )
   (wire (pts (xy 156.21 88.9) (xy 156.21 91.44))
     (stroke (width 0) (type default))
@@
     (stroke (width 0) (type default))
   )
+  (wire (pts (xy 69.85 63.5) (xy 69.85 64.77))
+    (stroke (width 0) (type default))
+  )
   (wire (pts (xy 156.21 85.09) (xy 158.75 85.09))
     (stroke (width 0) (type default))
@@
     (stroke (width 0) (type default))
   )
+  (wire (pts (xy 69.85 64.77) (xy 69.85 66.04))
+    (stroke (width 0) (type default))
+  )
   (wire (pts (xy 156.21 88.9) (xy 152.4 88.9))
     (stroke (width 0) (type default))
@@
   (wire (pts (xy 152.4 80.01) (xy 156.21 80.01))
     (stroke (width 0) (type default))
+  )
+  (label "EN" (at 76.2 64.77 180) (fields_autoplaced)
+    (effects (font (size 1.27 1.27)) (justify right bottom))
   )
   (label "EN" (at 120.65 90.17 0) (fields_autoplaced)
@@
     )
   )
+  (symbol (lib_id "Device:C_Small") (at 69.85 68.58 0) (mirror y) (unit 1)
+    (in_bom yes) (on_board yes) (dnp no)
+    (property "Reference" "C19" (at 67.5259 67.3742 0)
+      (effects (font (size 1.27 1.27)) (justify left))
+    )
+    (property "Value" "100nF" (at 67.5259 69.7984 0)
+      (effects (font (size 1.27 1.27)) (justify left))
+    )
+    (property "Footprint" "Capacitor_SMD:C_0402_1005Metric" (at 69.85 68.58 0)
+      (effects (font (size 1.27 1.27)) hide)
+    )
+    (property "Datasheet" "~" (at 69.85 68.58 0)
+      (effects (font (size 1.27 1.27)) hide)
+    )
+    (property "LCSC" "C1525" (at 69.85 68.58 0)
+      (effects (font (size 1.27 1.27)) hide)
+    )
+    (pin "1")
+    (pin "2")
+    (instances
+      (project "KASM_PCB_REV1"
+        (path "/bcd76057-59fd-41c5-bb52-9bafb2ef74e0/9f28d78d-ca42-4041-9be6-b996c46b4a0a"
+          (reference "C19") (unit 1)
+        )
+        (path "/bcd76057-59fd-41c5-bb52-9bafb2ef74e0/da6e1dd6-6549-4588-8765-3ff657cbe17b"
+          (reference "C1") (unit 1)
+        )
+        (path "/bcd76057-59fd-41c5-bb52-9bafb2ef74e0/04e958db-aa3d-41e7-905b-1283accbf3a5"
+          (reference "C37") (unit 1)
+        )
+        (path "/bcd76057-59fd-41c5-bb52-9bafb2ef74e0/04e958db-aa3d-41e7-905b-1283accbf3a5/317da025-5f62-4c93-8d06-7954e608af1c"
+          (reference "C37") (unit 1)
+        )
+        (path "/bcd76057-59fd-41c5-bb52-9bafb2ef74e0/04e958db-aa3d-41e7-905b-1283accbf3a5/09624144-9abc-4214-b8b3-19be92fa01bb"
+          (reference "C60") (unit 1)
+        )
+      )
+    )
+  )
+  (symbol (lib_id "power:+1V8") (at 69.85 58.42 0) (unit 1)
+    (in_bom yes) (on_board yes) (dnp no)
+    (property "Reference" "#PWR030" (at 69.85 62.23 0)
+      (effects (font (size 1.27 1.27)) hide)
+    )
+    (property "Value" "+1V8" (at 66.675 55.88 0)
+      (effects (font (size 1.27 1.27)))
+    )
+    (property "Footprint" "" (at 69.85 58.42 0)
+      (effects (font (size 1.27 1.27)) hide)
+    )
+    (property "Datasheet" "" (at 69.85 58.42 0)
+      (effects (font (size 1.27 1.27)) hide)
+    )
+    (pin "1")
+    (instances
+      (project "KASM_PCB_REV1"
+        (path "/bcd76057-59fd-41c5-bb52-9bafb2ef74e0/9f28d78d-ca42-4041-9be6-b996c46b4a0a"
+          (reference "#PWR030") (unit 1)
+        )
+        (path "/bcd76057-59fd-41c5-bb52-9bafb2ef74e0/04e958db-aa3d-41e7-905b-1283accbf3a5"
+          (reference "#PWR062") (unit 1)
+        )
+        (path "/bcd76057-59fd-41c5-bb52-9bafb2ef74e0/04e958db-aa3d-41e7-905b-1283accbf3a5/317da025-5f62-4c93-8d06-7954e608af1c"
+          (reference "#PWR014") (unit 1)
+        )
+        (path "/bcd76057-59fd-41c5-bb52-9bafb2ef74e0/04e958db-aa3d-41e7-905b-1283accbf3a5/09624144-9abc-4214-b8b3-19be92fa01bb"
+          (reference "#PWR0104") (unit 1)
+        )
+      )
+    )
+  )
   (symbol (lib_id "Device:R_Small_US") (at 156.21 106.68 0) (mirror y) (unit 1)
     (in_bom yes) (on_board yes) (dnp no)
@@
     )
   )
+  (symbol (lib_id "Device:R_Small_US") (at 69.85 60.96 0) (unit 1)
+    (in_bom yes) (on_board yes) (dnp no)
+    (property "Reference" "R23" (at 67.945 62.865 0)
+      (effects (font (size 1.27 1.27)) (justify right))
+    )
+    (property "Value" "10k" (at 68.58 60.325 0)
+      (effects (font (size 1.27 1.27)) (justify right))
+    )
+    (property "Footprint" "Resistor_SMD:R_0402_1005Metric" (at 69.85 60.96 0)
+      (effects (font (size 1.27 1.27)) hide)
+    )
+    (property "Datasheet" "~" (at 69.85 60.96 0)
+      (effects (font (size 1.27 1.27)) hide)
+    )
+    (property "LCSC" "C25744" (at 69.85 60.96 0)
+      (effects (font (size 1.27 1.27)) hide)
+    )
+    (pin "1")
+    (pin "2")
+    (instances
+      (project "KASM_PCB_REV1"
+        (path "/bcd76057-59fd-41c5-bb52-9bafb2ef74e0/04e958db-aa3d-41e7-905b-1283accbf3a5"
+          (reference "R23") (unit 1)
+        )
+        (path "/bcd76057-59fd-41c5-bb52-9bafb2ef74e0/04e958db-aa3d-41e7-905b-1283accbf3a5/317da025-5f62-4c93-8d06-7954e608af1c"
+          (reference "R23") (unit 1)
+        )
+        (path "/bcd76057-59fd-41c5-bb52-9bafb2ef74e0/04e958db-aa3d-41e7-905b-1283accbf3a5/09624144-9abc-4214-b8b3-19be92fa01bb"
+          (reference "R44") (unit 1)
+        )
+      )
+    )
+  )
   (symbol (lib_id "power:GND") (at 156.21 110.49 0) (unit 1)
     (in_bom yes) (on_board yes) (dnp no)
@@
         )
       )
+    )
+  )
+  (symbol (lib_id "power:GND") (at 69.85 72.39 0) (unit 1)
+    (in_bom yes) (on_board yes) (dnp no)
+    (property "Reference" "#PWR064" (at 69.85 78.74 0)
+      (effects (font (size 1.27 1.27)) hide)
+    )
+    (property "Value" "GND" (at 69.85 76.5231 0)
+      (effects (font (size 1.27 1.27)))
+    )
+    (property "Footprint" "" (at 69.85 72.39 0)
+      (effects (font (size 1.27 1.27)) hide)
+    )
+    (property "Datasheet" "" (at 69.85 72.39 0)
+      (effects (font (size 1.27 1.27)) hide)
+    )
+    (pin "1")
+    (instances
+      (project "KASM_PCB_REV1"
+        (path "/bcd76057-59fd-41c5-bb52-9bafb2ef74e0/04e958db-aa3d-41e7-905b-1283accbf3a5"
+          (reference "#PWR064") (unit 1)
+        )
+        (path "/bcd76057-59fd-41c5-bb52-9bafb2ef74e0/04e958db-aa3d-41e7-905b-1283accbf3a5/317da025-5f62-4c93-8d06-7954e608af1c"
+          (reference "#PWR015") (unit 1)
+        )
+        (path "/bcd76057-59fd-41c5-bb52-9bafb2ef74e0/04e958db-aa3d-41e7-905b-1283accbf3a5/09624144-9abc-4214-b8b3-19be92fa01bb"
+          (reference "#PWR0105") (unit 1)
+        )
+      )

Commit message: Add files via upload
Parts:
- C19: value 100nF -> 10nF; LCSC C1525 -> C15195
- R31: value 1.4R -> 1.0R; LCSC C305315 -> C17928
Changed lines of the file:
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@@
       (effects (font (size 1.27 1.27)) (justify left))
     )
-    (property "Value" "100nF" (at 67.5259 69.7984 0)
+    (property "Value" "10nF" (at 67.5259 69.7984 0)
       (effects (font (size 1.27 1.27)) (justify left))
     )
@@
       (effects (font (size 1.27 1.27)) hide)
     )
-    (property "LCSC" "C1525" (at 69.85 68.58 0)
+    (property "LCSC" "C15195" (at 69.85 68.58 0)
       (effects (font (size 1.27 1.27)) hide)
     )
@@
       (effects (font (size 1.27 1.27)) (justify right))
     )
-    (property "Value" "1.4R" (at 157.861 107.8921 0)
+    (property "Value" "1.0R" (at 157.861 107.8921 0)
       (effects (font (size 1.27 1.27)) (justify right))
     )
@@
       (effects (font (size 1.27 1.27)) hide)
     )
-    (property "LCSC" "C305315" (at 156.21 106.68 0)
+    (property "LCSC" "C17928" (at 156.21 106.68 0)
       (effects (font (size 1.27 1.27)) hide)
     )
