File: KASM_PCB_REV1_MCU.kicad_sch (KiCad schematic)
At the start: 39 parts, among them J1 Conn_01x06, J3 Conn_01x03, J31 Conn_01x05, J32 Conn_01x02, J33 Conn_01x02, SW1 SW_Push, U1 STM32H750VBTx, U29 TLV9062xD, U5 TLV9062xD, U6 M24C02-WMN, Y1 24MHz, 9pF

Commit message: Add files via upload
Parts:
- removed C11: 2.2uF, symbol Device:C_Small
- removed C3: 100nF, symbol Device:C_Small
- removed U29, U5: TLV9062xD, Package_SO:SOIC-8_3.9x4.9mm_P1.27mm, symbol Amplifier_Operational:TLV9062xD
- added C19: 100nF, Capacitor_SMD:C_0402_1005Metric, symbol Device:C_Small
- added C8: 2.2uF, Capacitor_SMD:C_0402_1005Metric, symbol Device:C_Small
- added R2: 10k, Resistor_SMD:R_0402_1005Metric, symbol Device:R_US
- added SW1: SW_Push, Button_Switch_SMD:SW_Push_1P1T_XKB_TS-1187A, symbol Switch:SW_Push
- added U4: TLV9062xD, Package_SO:SOIC-8_3.9x4.9mm_P1.27mm, symbol Amplifier_Operational:TLV9062xD
- C8: footprint (none) -> Capacitor_SMD:C_0402_1005Metric; LCSC (none) -> C12530
- C9: footprint (none) -> Capacitor_SMD:C_0402_1005Metric; LCSC (none) -> C23733
- J5: renamed from J1; footprint (none) -> Connector_PinHeader_2.54mm:PinHeader_1x06_P2.54mm_Vertical
- J6: renamed from J31; footprint (none) -> Connector_PinHeader_2.54mm:PinHeader_1x05_P2.54mm_Vertical
- J7: renamed from J3; footprint (none) -> Connector_PinHeader_2.54mm:PinHeader_1x03_P2.54mm_Vertical
- SW1: LCSC (none) -> C318884
- U3: renamed from U6; LCSC (none) -> C7562
- renumbered J32 to J3, J33 to J4, R13 to R12, R1 to R13, R17 to R14, R16 to R15, R15 to R16, R14 to R17, R102 to R18, R104 to R19, R105 to R20, R106 to R21, R103 to R22
Connections:
- net +3.3V: now also C19.1, SW1.2, U4.4 (V-)
- net ADC1_INP4: now also U4.1
- net ADC1_INP5: now also U4.7
- net BOOT0: now also R2.1, SW1.1
- net GND: now also C19.2, C8.2, R2.2, U4.8 (V+)
- net HRTIM_CHB1: no longer U1.79 (PC11)
- net UART4_RX: now also U1.79 (PC11); no longer U1.66 (PC9)
- net at R19.2, R20.1: now also U4.6 (-)
- net at R21.1, R22.1: now also U4.5 (+)
- net at U1.73 (VCAP): now also C8.1
- net at R14.2, R16.1: now also U4.2 (-)
- net at R17.1, R18.1: now also U4.3 (+)
- new net TIM8_CH4: U1.66 (PC9)
- no-connect marks 1 -> 13
Other:
- moved on the sheet: J6

Commit message: Add files via upload
Parts:
- removed C1: 10uF, Capacitor_SMD:C_1206_3216Metric, symbol Device:C_Small
- added C9: 4.7uF, Capacitor_SMD:C_0402_1005Metric, symbol Device:C_Small
Connections:
- net GND: now also C9.1
- net VREF+: now also C9.2
Changed lines of the file:
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@@
-    )
-  )
-  (symbol (lib_id "Device:C_Small") (at 246.38 78.74 0) (unit 1)
-    (in_bom yes) (on_board yes) (dnp no) (fields_autoplaced)
-    (property "Reference" "C1" (at 248.7041 77.5342 0)
-      (effects (font (size 1.27 1.27)) (justify left))
-    )
-    (property "Value" "10uF" (at 248.7041 79.9584 0)
-      (effects (font (size 1.27 1.27)) (justify left))
-    )
-    (property "Footprint" "Capacitor_SMD:C_1206_3216Metric" (at 246.38 78.74 0)
-      (effects (font (size 1.27 1.27)) hide)
-    )
-    (property "Datasheet" "~" (at 246.38 78.74 0)
-      (effects (font (size 1.27 1.27)) hide)
-    )
-    (property "LCSC" "C454102" (at 246.38 78.74 0)
-      (effects (font (size 1.27 1.27)) hide)
-    )
-    (pin "1")
-    (pin "2")
-    (instances
-      (project "KASM_PCB_REV1"
-        (path "/bcd76057-59fd-41c5-bb52-9bafb2ef74e0"
-          (reference "C1") (unit 1)
-        )
-        (path "/bcd76057-59fd-41c5-bb52-9bafb2ef74e0/da6e1dd6-6549-4588-8765-3ff657cbe17b"
-          (reference "C30") (unit 1)
-        )
-      )
     )
   )
@@
         )
       )
+    )
+  )
+  (symbol (lib_id "Device:C_Small") (at 246.38 78.74 180) (unit 1)
+    (in_bom yes) (on_board yes) (dnp no)
+    (property "Reference" "C9" (at 248.7041 77.5215 0)
+      (effects (font (size 1.27 1.27)) (justify right))
+    )
+    (property "Value" "4.7uF" (at 248.7041 79.9457 0)
+      (effects (font (size 1.27 1.27)) (justify right))
+    )
+    (property "Footprint" "Capacitor_SMD:C_0402_1005Metric" (at 246.38 78.74 0)
+      (effects (font (size 1.27 1.27)) hide)
+    )
+    (property "Datasheet" "~" (at 246.38 78.74 0)
+      (effects (font (size 1.27 1.27)) hide)
+    )
+    (property "LCSC" "C23733" (at 246.38 78.74 0)
+      (effects (font (size 1.27 1.27)) hide)
+    )
+    (pin "1")
+    (pin "2")
+    (instances
+      (project "KASM_PCB_REV1"
+        (path "/bcd76057-59fd-41c5-bb52-9bafb2ef74e0"
+          (reference "C9") (unit 1)
+        )
+        (path "/bcd76057-59fd-41c5-bb52-9bafb2ef74e0/da6e1dd6-6549-4588-8765-3ff657cbe17b"
+          (reference "C30") (unit 1)
+        )
+      )

Commit message: Add files via upload
Connections:
- net HRTIM_CHD2: no longer U1.71 (PA12)
Other:
- note added: "CAPACITIVE SENSOR ANALOG"
- note removed: "Capacitive Sensors"
Changed lines of the file:
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@@
-    (stroke (width 0) (type default))
-  )
-  (wire (pts (xy 250.19 109.22) (xy 245.11 109.22))
     (stroke (width 0) (type default))
   )
@@
     (stroke (width 0) (type default))
   )
+  (wire (pts (xy 245.11 96.52) (xy 250.19 96.52))
+    (stroke (width 0) (type default))
+  )
   (wire (pts (xy 342.9 132.08) (xy 342.9 133.35))
     (stroke (width 0) (type default))
@@
     (stroke (width 0) (type default))
   )
-  (wire (pts (xy 250.19 93.98) (xy 245.11 93.98))
-    (stroke (width 0) (type default))
-  )
   (wire (pts (xy 193.04 44.45) (xy 193.04 45.72))
     (stroke (width 0) (type default))
@@
     (stroke (width 0) (type default))
   )
+  (wire (pts (xy 248.92 121.92) (xy 245.11 121.92))
+    (stroke (width 0) (type default))
+  )
   (wire (pts (xy 196.85 180.34) (xy 201.93 180.34))
     (stroke (width 0) (type default))
@@
     (stroke (width 0) (type default))
   )
-  (wire (pts (xy 250.19 96.52) (xy 245.11 96.52))
-    (stroke (width 0) (type default))
-  )
   (wire (pts (xy 250.19 187.96) (xy 245.11 187.96))
     (stroke (width 0) (type default))
@@
     (stroke (width 0) (type default))
   )
+  (wire (pts (xy 245.11 91.44) (xy 250.19 91.44))
+    (stroke (width 0) (type default))
+  )
   (wire (pts (xy 222.25 82.55) (xy 224.79 82.55))
     (stroke (width 0) (type default))
@@
     (stroke (width 0) (type default))
   )
-  (wire (pts (xy 250.19 119.38) (xy 245.11 119.38))
-    (stroke (width 0) (type default))
-  )
   (wire (pts (xy 250.19 180.34) (xy 245.11 180.34))
     (stroke (width 0) (type default))
@@
     (stroke (width 0) (type default))
   )
-  (wire (pts (xy 250.19 116.84) (xy 245.11 116.84))
+  (wire (pts (xy 245.11 116.84) (xy 250.19 116.84))
     (stroke (width 0) (type default))
   )
@@
     (stroke (width 0) (type default))
   )
-  (wire (pts (xy 250.19 106.68) (xy 245.11 106.68))
-    (stroke (width 0) (type default))
-  )
   (wire (pts (xy 160.02 49.53) (xy 160.02 50.8))
     (stroke (width 0) (type default))
@@
     (stroke (width 0) (type default))
   )
+  (wire (pts (xy 245.11 109.22) (xy 250.19 109.22))
+    (stroke (width 0) (type default))
+  )
   (wire (pts (xy 222.25 226.06) (xy 222.25 227.33))
     (stroke (width 0) (type default))
   )
+  (wire (pts (xy 245.11 93.98) (xy 250.19 93.98))
+    (stroke (width 0) (type default))
+  )
   (wire (pts (xy 204.47 53.34) (xy 215.9 53.34))
     (stroke (width 0) (type default))
@@
     (stroke (width 0) (type default))
   )
-  (wire (pts (xy 250.19 111.76) (xy 245.11 111.76))
+  (wire (pts (xy 245.11 111.76) (xy 250.19 111.76))
     (stroke (width 0) (type default))
   )
@@
     (stroke (width 0) (type default))
   )
-  (wire (pts (xy 250.19 91.44) (xy 245.11 91.44))
-    (stroke (width 0) (type default))
-  )
   (wire (pts (xy 97.79 102.87) (xy 97.79 113.03))
     (stroke (width 0) (type default))
@@
     (stroke (width 0) (type default))
   )
+  (wire (pts (xy 245.11 114.3) (xy 250.19 114.3))
+    (stroke (width 0) (type default))
+  )
   (wire (pts (xy 222.25 227.33) (xy 222.25 228.6))
     (stroke (width 0) (type default))
@@
     (stroke (width 0) (type default))
   )
+  (wire (pts (xy 245.11 119.38) (xy 250.19 119.38))
+    (stroke (width 0) (type default))
+  )
   (wire (pts (xy 196.85 160.02) (xy 201.93 160.02))
     (stroke (width 0) (type default))
@@
     (stroke (width 0) (type default))
   )
-  (wire (pts (xy 250.19 121.92) (xy 245.11 121.92))
+  (wire (pts (xy 250.19 121.92) (xy 256.54 121.92))
     (stroke (width 0) (type default))
   )
@@
     (stroke (width 0) (type default))
   )
+  (wire (pts (xy 245.11 106.68) (xy 250.19 106.68))
+    (stroke (width 0) (type default))
+  )
   (wire (pts (xy 334.01 48.26) (xy 334.01 49.53))
     (stroke (width 0) (type default))
@@
     (stroke (width 0) (type default))
   )
-  (wire (pts (xy 250.19 114.3) (xy 245.11 114.3))
-    (stroke (width 0) (type default))
-  )
   (wire (pts (xy 217.17 82.55) (xy 217.17 83.82))
     (stroke (width 0) (type default))
@@
     (fill (type none))
   )
-  (text "Capacitive Sensors" (at 45.72 52.07 0)
+  (text "CAPACITIVE SENSOR ANALOG" (at 31.75 52.07 0)
     (effects (font (size 5 5)) (justify left bottom))
   )

Commit message: Add files via upload
Connections:
- net HRTIM_CHD2: now also U1.71 (PA12)
Changed lines of the file:
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@@
     (stroke (width 0) (type default))
   )
-  (wire (pts (xy 248.92 121.92) (xy 245.11 121.92))
+  (wire (pts (xy 245.11 121.92) (xy 250.19 121.92))
     (stroke (width 0) (type default))
   )
@@
     (stroke (width 0) (type default))
   )
-  (wire (pts (xy 250.19 121.92) (xy 256.54 121.92))
-    (stroke (width 0) (type default))
-  )

Commit message: Add files via upload
Parts:
- U4: LCSC (none) -> C398355
Changed lines of the file:
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@@
+      (effects (font (size 1.27 1.27)) hide)
+    )
+    (property "LCSC" "C398355" (at 88.9 113.03 0)
       (effects (font (size 1.27 1.27)) hide)
     )
@@
       (effects (font (size 1.27 1.27)) hide)
     )
+    (property "LCSC" "C398355" (at 88.9 152.4 0)
+      (effects (font (size 1.27 1.27)) hide)
+    )
     (pin "1")
     (pin "2")
@@
       (effects (font (size 1.27 1.27)) hide)
     )
+    (property "LCSC" "C398355" (at 100.33 74.93 0)
+      (effects (font (size 1.27 1.27)) hide)
+    )

Commit message: Add files via upload
Parts:
- added C18 (x4): 2.2nF, Capacitor_SMD:C_0402_1005Metric, symbol Device:C_Small
- R16, R17, R20, R21: LCSC C25105 -> C25779
Connections:
- net ADC1_INP4: now also C18.2
- net ADC1_INP5: now also C18.1
- net GND: now also C18.1, C18.1
- net at R14.2, R16.1, U4.2 (-): now also C18.1
- net at R17.1, R18.1, U4.3 (+): now also C18.2
- net at R19.2, R20.1, U4.6 (-): now also C18.2
- net at R21.1, R22.1, U4.5 (+): now also C18.2
Other:
- moved on the sheet: R14, R19

Commit message: Add files via upload
Parts:
- added TP1, TP2, TP3, TP4, TP5: TestPoint, TestPoint:TestPoint_Pad_1.0x1.0mm, symbol Connector:TestPoint
Connections:
- net ADC2_INP10: now reaches U1.15 (PC0)
- net ADC2_INP10: now also TP5.1
- net ADC1_INP15: now reaches U1.25 (PA3)
- net ADC1_INP15: now also TP1.1
- net ADC1_INP18: now reaches U1.28 (PA4)
- net ADC1_INP18: now also TP2.1
- net ADC1_INP19: now reaches U1.29 (PA5)
- net ADC1_INP19: now also TP3.1
- net ADC2_INP9: now reaches U1.34 (PB0)
- net ADC2_INP9: now also TP4.1
- no-connect marks 13 -> 8
Other:
- note added: "TEST POINTS"
